File: uSensor_v1/Coil_Current_Source.sch (KiCad schematic (older format))
At the start: 14 parts, among them Q3 BC847PN-7-F, U17 TBD

Commit message: Schematic changed (added 2channel opamp in one HS)
Parts:
- removed C54, C55: 100n 6V3 X5R, Capacitor_SMD:C_0603_1608Metric_Pad1.05x0.95mm_HandSolder, symbol Device:C
- removed Q3: BC847PN-7-F, Sentisa-IC:SOT-363, symbol Transistor_BJT:BC847BPDW1
- removed R38, R44: 1R, Resistor_SMD:R_0603_1608Metric_Pad1.05x0.95mm_HandSolder, symbol Device:R
- removed R39, R40, R42: 10k 1%, Resistor_SMD:R_0603_1608Metric_Pad1.05x0.95mm_HandSolder, symbol Device:R
- removed R41: 10k, Resistor_SMD:R_0603_1608Metric_Pad1.05x0.95mm_HandSolder, symbol Device:R
- removed R43: 10R, Resistor_SMD:R_0603_1608Metric_Pad1.05x0.95mm_HandSolder, symbol Device:R
- removed RV3: 20k, Sentisa-Resistors:Potentiometer_SR_Passives_T910W_Vertical, symbol Device:R_POT
- removed TP79, TP80: TP, Sentisa-Connectors:TestPoint_Probe_1.0mmDiameter_0.6mmDrill, symbol Connector:TestPoint
- removed U17: TBD, TBD, symbol Amplifier_Operational:LM321
Connections:
- net labels removed: COIL+, COIL-, DAC_IN, GND, PWR_IN+, PWR_IN-
- wire segments 50 -> 0
