File: uSensor_v1/SENS_IN_AMP.sch (KiCad schematic (older format))
At the start: 8 parts

Commit message: Schematic in progress.
Other:
- moved on the sheet: C?
Changed lines of the file:
@@
 $Descr A4 11693 8268
 encoding utf-8
-Sheet 2 5
+Sheet 4 5
 Title ""
 Date ""
@@
 L Device:C C?
 U 1 1 5C6F020C
-P 5300 2750
+P 5300 2650
 AR Path="/5C6F020C" Ref="C?"  Part="1"
 AR Path="/5C6EFF05/5C6F020C" Ref="C?"  Part="1"
@@
 AR Path="/5C829D40/5C6F020C" Ref="C?"  Part="1"
 AR Path="/5C7ECB16/5C6F020C" Ref="C?"  Part="1"
-F 0 "C?" H 5415 2796 50  0000 L CNN
-F 1 "1p" H 5415 2705 50  0000 L CNN
-F 2 "" H 5338 2600 50  0001 C CNN
-F 3 "~" H 5300 2750 50  0001 C CNN
-	1    5300 2750
+F 0 "C?" H 5415 2696 50  0000 L CNN
+F 1 "1p" H 5415 2605 50  0000 L CNN
+F 2 "" H 5338 2500 50  0001 C CNN
+F 3 "~" H 5300 2650 50  0001 C CNN
+	1    5300 2650
 	0    1    1    0
 $EndComp
@@
 $EndComp
 Wire Wire Line
-	5450 2750 5450 2850
+	5450 2650 5450 2850
 Connection ~ 5150 2850
 Wire Wire Line
@@
 	5000 3300 4900 3300
 Wire Wire Line
-	5150 2750 5150 2850
+	5150 2650 5150 2850
 Wire Wire Line
 	5000 2850 5150 2850
@@
 AR Path="/5C86721C/5C6F023D" Ref="#PWR?"  Part="1"
 AR Path="/5C829D40/5C6F023D" Ref="#PWR?"  Part="1"
+AR Path="/5C7ECB16/5C6F023D" Ref="#PWR?"  Part="1"
 F 0 "#PWR?" H 4950 3850 50  0001 C CNN
 F 1 "GND" H 4955 3927 50  0000 C CNN
@@
 AR Path="/5C86721C/5C6F0247" Ref="#PWR?"  Part="1"
 AR Path="/5C829D40/5C6F0247" Ref="#PWR?"  Part="1"
+AR Path="/5C7ECB16/5C6F0247" Ref="#PWR?"  Part="1"
 F 0 "#PWR?" H 6000 4050 50  0001 C CNN
 F 1 "-5V" V 6015 4078 50  0000 L CNN
@@
 AR Path="/5C86721C/5C6F024D" Ref="#PWR?"  Part="1"
 AR Path="/5C829D40/5C6F024D" Ref="#PWR?"  Part="1"
+AR Path="/5C7ECB16/5C6F024D" Ref="#PWR?"  Part="1"
 F 0 "#PWR?" H 6000 2600 50  0001 C CNN
 F 1 "+5V" V 6015 2878 50  0000 L CNN
@@
 AR Path="/5C86721C/5C6F025A" Ref="#PWR?"  Part="1"
 AR Path="/5C829D40/5C6F025A" Ref="#PWR?"  Part="1"
+AR Path="/5C7ECB16/5C6F025A" Ref="#PWR?"  Part="1"
 F 0 "#PWR?" H 6000 2800 50  0001 C CNN
 F 1 "GND" H 6005 2877 50  0000 C CNN
@@
 AR Path="/5C86721C/5C6F0260" Ref="C?"  Part="1"
 AR Path="/5C829D40/5C6F0260" Ref="C?"  Part="1"
+AR Path="/5C7ECB16/5C6F0260" Ref="C?"  Part="1"
 F 0 "C?" H 6115 4146 50  0000 L CNN
 F 1 "100n 6V3 X5R" H 6115 4055 50  0000 L CNN
@@
 AR Path="/5C86721C/5C6F0267" Ref="#PWR?"  Part="1"
 AR Path="/5C829D40/5C6F0267" Ref="#PWR?"  Part="1"
+AR Path="/5C7ECB16/5C6F0267" Ref="#PWR?"  Part="1"
 F 0 "#PWR?" H 6000 4000 50  0001 C CNN
 F 1 "GND" H 6005 4077 50  0000 C CNN

Commit message: Schematic in progress.
Parts:
- U?: footprint Package_TO_SOT_SMD:TSOT-23-5 -> (none)
Changed lines of the file:
@@
 F 0 "U?" H 5500 3650 50  0000 L CNN
 F 1 "LM6132A/NS" H 5650 3650 50  0000 L CNN
-F 2 "Package_TO_SOT_SMD:TSOT-23-5" H 5400 3550 50  0001 C CNN
+F 2 "" H 5400 3550 50  0001 C CNN
 F 3 "http://www.analog.com/media/en/technical-documentation/data-sheets/AD8603_8607_8609.pdf" H 5400 3750 50  0001 C CNN
 	1    5400 3550
@@
 AR Path="/5C86721C/5C6F0253" Ref="C?"  Part="1"
 AR Path="/5C829D40/5C6F0253" Ref="C?"  Part="1"
+AR Path="/5C7ECB16/5C6F0253" Ref="C?"  Part="1"
 F 0 "C?" H 6115 2946 50  0000 L CNN
 F 1 "100n 6V3 X5R" H 6115 2855 50  0000 L CNN

Commit message: Schematic in progress.
Parts:
- C? (x3): footprint (none) -> Capacitor_SMD:C_0603_1608Metric_Pad1.05x0.95mm_HandSolder
Connections:
- net +5V renamed PWR_IN+
- net -5V renamed PWR_IN-
Other:
- moved on the sheet: C?, R?

Commit message: Schematic in progress.
Parts:
- gave numbers to parts that had none: 8
Changed lines of the file:
@@
 P 5400 3550
 AR Path="/5C6F01FE" Ref="U?"  Part="1"
-AR Path="/5C6EFF05/5C6F01FE" Ref="U?"  Part="1"
+AR Path="/5C6EFF05/5C6F01FE" Ref="U16"  Part="1"
 AR Path="/5C86721C/5C6F01FE" Ref="U?"  Part="1"
 AR Path="/5C829D40/5C6F01FE" Ref="U?"  Part="1"
 AR Path="/5C7ECB16/5C6F01FE" Ref="U?"  Part="1"
-AR Path="/5D09CD82/5C6F01FE" Ref="U?"  Part="1"
-AR Path="/5D0DF15B/5C6F01FE" Ref="U?"  Part="1"
-AR Path="/5D1213F6/5C6F01FE" Ref="U?"  Part="1"
-F 0 "U?" H 5500 3650 50  0000 L CNN
+AR Path="/5D09CD82/5C6F01FE" Ref="U19"  Part="1"
+AR Path="/5D0DF15B/5C6F01FE" Ref="U20"  Part="1"
+AR Path="/5D1213F6/5C6F01FE" Ref="U21"  Part="1"
+F 0 "U21" H 5500 3650 50  0000 L CNN
 F 1 "LM6132A/NS" H 5400 3350 50  0000 L CNN
 F 2 "" H 5400 3550 50  0001 C CNN
@@
 P 4450 3650
 AR Path="/5C6F0205" Ref="R?"  Part="1"
-AR Path="/5C6EFF05/5C6F0205" Ref="R?"  Part="1"
+AR Path="/5C6EFF05/5C6F0205" Ref="R36"  Part="1"
 AR Path="/5C86721C/5C6F0205" Ref="R?"  Part="1"
 AR Path="/5C829D40/5C6F0205" Ref="R?"  Part="1"
 AR Path="/5C7ECB16/5C6F0205" Ref="R?"  Part="1"
-AR Path="/5D09CD82/5C6F0205" Ref="R?"  Part="1"
-AR Path="/5D0DF15B/5C6F0205" Ref="R?"  Part="1"
-AR Path="/5D1213F6/5C6F0205" Ref="R?"  Part="1"
-F 0 "R?" V 4243 3650 50  0000 C CNN
+AR Path="/5D09CD82/5C6F0205" Ref="R54"  Part="1"
+AR Path="/5D0DF15B/5C6F0205" Ref="R58"  Part="1"
+AR Path="/5D1213F6/5C6F0205" Ref="R62"  Part="1"
+F 0 "R62" V 4243 3650 50  0000 C CNN
 F 1 "10k" V 4334 3650 50  0000 C CNN
 F 2 "" V 4380 3650 50  0001 C CNN
@@
 P 5350 2500
 AR Path="/5C6F020C" Ref="C?"  Part="1"
-AR Path="/5C6EFF05/5C6F020C" Ref="C?"  Part="1"
+AR Path="/5C6EFF05/5C6F020C" Ref="C51"  Part="1"
 AR Path="/5C86721C/5C6F020C" Ref="C?"  Part="1"
 AR Path="/5C829D40/5C6F020C" Ref="C?"  Part="1"
 AR Path="/5C7ECB16/5C6F020C" Ref="C?"  Part="1"
-AR Path="/5D09CD82/5C6F020C" Ref="C?"  Part="1"
-AR Path="/5D0DF15B/5C6F020C" Ref="C?"  Part="1"
-AR Path="/5D1213F6/5C6F020C" Ref="C?"  Part="1"
-F 0 "C?" V 5098 2500 50  0000 C CNN
+AR Path="/5D09CD82/5C6F020C" Ref="C58"  Part="1"
+AR Path="/5D0DF15B/5C6F020C" Ref="C61"  Part="1"
+AR Path="/5D1213F6/5C6F020C" Ref="C64"  Part="1"
+F 0 "C64" V 5098 2500 50  0000 C CNN
 F 1 "1p" V 5189 2500 50  0000 C CNN
 F 2 "Capacitor_SMD:C_0603_1608Metric_Pad1.05x0.95mm_HandSolder" H 5388 2350 50  0001 C CNN
@@
 P 4700 3900
 AR Path="/5C6F0213" Ref="R?"  Part="1"
-AR Path="/5C6EFF05/5C6F0213" Ref="R?"  Part="1"
+AR Path="/5C6EFF05/5C6F0213" Ref="R37"  Part="1"
 AR Path="/5C86721C/5C6F0213" Ref="R?"  Part="1"
 AR Path="/5C829D40/5C6F0213" Ref="R?"  Part="1"
 AR Path="/5C7ECB16/5C6F0213" Ref="R?"  Part="1"
-AR Path="/5D09CD82/5C6F0213" Ref="R?"  Part="1"
-AR Path="/5D0DF15B/5C6F0213" Ref="R?"  Part="1"
-AR Path="/5D1213F6/5C6F0213" Ref="R?"  Part="1"
-F 0 "R?" H 4770 3946 50  0000 L CNN
+AR Path="/5D09CD82/5C6F0213" Ref="R55"  Part="1"
+AR Path="/5D0DF15B/5C6F0213" Ref="R59"  Part="1"
+AR Path="/5D1213F6/5C6F0213" Ref="R63"  Part="1"
+F 0 "R63" H 4770 3946 50  0000 L CNN
 F 1 "22k" H 4770 3855 50  0000 L CNN
 F 2 "" V 4630 3900 50  0001 C CNN
@@
 P 4450 3300
 AR Path="/5C6F0221" Ref="R?"  Part="1"
-AR Path="/5C6EFF05/5C6F0221" Ref="R?"  Part="1"
+AR Path="/5C6EFF05/5C6F0221" Ref="R35"  Part="1"
 AR Path="/5C86721C/5C6F0221" Ref="R?"  Part="1"
 AR Path="/5C829D40/5C6F0221" Ref="R?"  Part="1"
 AR Path="/5C7ECB16/5C6F0221" Ref="R?"  Part="1"
-AR Path="/5D09CD82/5C6F0221" Ref="R?"  Part="1"
-AR Path="/5D0DF15B/5C6F0221" Ref="R?"  Part="1"
-AR Path="/5D1213F6/5C6F0221" Ref="R?"  Part="1"
-F 0 "R?" V 4243 3300 50  0000 C CNN
+AR Path="/5D09CD82/5C6F0221" Ref="R53"  Part="1"
+AR Path="/5D0DF15B/5C6F0221" Ref="R57"  Part="1"
+AR Path="/5D1213F6/5C6F0221" Ref="R61"  Part="1"
+F 0 "R61" V 4243 3300 50  0000 C CNN
 F 1 "10k" V 4334 3300 50  0000 C CNN
 F 2 "" V 4380 3300 50  0001 C CNN
@@
 P 5350 2850
 AR Path="/5C6F0228" Ref="R?"  Part="1"
-AR Path="/5C6EFF05/5C6F0228" Ref="R?"  Part="1"
+AR Path="/5C6EFF05/5C6F0228" Ref="R34"  Part="1"
 AR Path="/5C86721C/5C6F0228" Ref="R?"  Part="1"
 AR Path="/5C829D40/5C6F0228" Ref="R?"  Part="1"
 AR Path="/5C7ECB16/5C6F0228" Ref="R?"  Part="1"
-AR Path="/5D09CD82/5C6F0228" Ref="R?"  Part="1"
-AR Path="/5D0DF15B/5C6F0228" Ref="R?"  Part="1"
-AR Path="/5D1213F6/5C6F0228" Ref="R?"  Part="1"
-F 0 "R?" V 5143 2850 50  0000 C CNN
+AR Path="/5D09CD82/5C6F0228" Ref="R52"  Part="1"
+AR Path="/5D0DF15B/5C6F0228" Ref="R56"  Part="1"
+AR Path="/5D1213F6/5C6F0228" Ref="R60"  Part="1"
+F 0 "R60" V 5143 2850 50  0000 C CNN
 F 1 "22k" V 5234 2850 50  0000 C CNN
 F 2 "" V 5280 2850 50  0001 C CNN
@@
 P 6000 2750
 AR Path="/5C6F0253" Ref="C?"  Part="1"
-AR Path="/5C6EFF05/5C6F0253" Ref="C?"  Part="1"
+AR Path="/5C6EFF05/5C6F0253" Ref="C52"  Part="1"
 AR Path="/5C86721C/5C6F0253" Ref="C?"  Part="1"
 AR Path="/5C829D40/5C6F0253" Ref="C?"  Part="1"
 AR Path="/5C7ECB16/5C6F0253" Ref="C?"  Part="1"
-AR Path="/5D09CD82/5C6F0253" Ref="C?"  Part="1"
-AR Path="/5D0DF15B/5C6F0253" Ref="C?"  Part="1"
-AR Path="/5D1213F6/5C6F0253" Ref="C?"  Part="1"
-F 0 "C?" H 6115 2796 50  0000 L CNN
+AR Path="/5D09CD82/5C6F0253" Ref="C59"  Part="1"
+AR Path="/5D0DF15B/5C6F0253" Ref="C62"  Part="1"
+AR Path="/5D1213F6/5C6F0253" Ref="C65"  Part="1"
+F 0 "C65" H 6115 2796 50  0000 L CNN
 F 1 "100n 6V3 X5R" H 6115 2705 50  0000 L CNN
 F 2 "Capacitor_SMD:C_0603_1608Metric_Pad1.05x0.95mm_HandSolder" H 6038 2600 50  0001 C CNN
@@
 P 6000 4500
 AR Path="/5C6F0260" Ref="C?"  Part="1"
-AR Path="/5C6EFF05/5C6F0260" Ref="C?"  Part="1"
+AR Path="/5C6EFF05/5C6F0260" Ref="C53"  Part="1"
 AR Path="/5C86721C/5C6F0260" Ref="C?"  Part="1"
 AR Path="/5C829D40/5C6F0260" Ref="C?"  Part="1"
 AR Path="/5C7ECB16/5C6F0260" Ref="C?"  Part="1"
-AR Path="/5D09CD82/5C6F0260" Ref="C?"  Part="1"
-AR Path="/5D0DF15B/5C6F0260" Ref="C?"  Part="1"
-AR Path="/5D1213F6/5C6F0260" Ref="C?"  Part="1"
-F 0 "C?" H 6115 4546 50  0000 L CNN
+AR Path="/5D09CD82/5C6F0260" Ref="C60"  Part="1"
+AR Path="/5D0DF15B/5C6F0260" Ref="C63"  Part="1"
+AR Path="/5D1213F6/5C6F0260" Ref="C66"  Part="1"
+F 0 "C66" H 6115 4546 50  0000 L CNN
 F 1 "100n 6V3 X5R" H 6115 4455 50  0000 L CNN
 F 2 "Capacitor_SMD:C_0603_1608Metric_Pad1.05x0.95mm_HandSolder" H 6038 4350 50  0001 C CNN

Commit message: Schematic in progress.
Changed lines of the file:
@@
 AR Path="/5D0DF15B/5C6F01FE" Ref="U20"  Part="1"
 AR Path="/5D1213F6/5C6F01FE" Ref="U21"  Part="1"
-F 0 "U21" H 5500 3650 50  0000 L CNN
+F 0 "U16" H 5500 3650 50  0000 L CNN
 F 1 "LM6132A/NS" H 5400 3350 50  0000 L CNN
 F 2 "" H 5400 3550 50  0001 C CNN
@@
 AR Path="/5D0DF15B/5C6F0205" Ref="R58"  Part="1"
 AR Path="/5D1213F6/5C6F0205" Ref="R62"  Part="1"
-F 0 "R62" V 4243 3650 50  0000 C CNN
+F 0 "R36" V 4243 3650 50  0000 C CNN
 F 1 "10k" V 4334 3650 50  0000 C CNN
 F 2 "" V 4380 3650 50  0001 C CNN
@@
 AR Path="/5D0DF15B/5C6F020C" Ref="C61"  Part="1"
 AR Path="/5D1213F6/5C6F020C" Ref="C64"  Part="1"
-F 0 "C64" V 5098 2500 50  0000 C CNN
+F 0 "C51" V 5098 2500 50  0000 C CNN
 F 1 "1p" V 5189 2500 50  0000 C CNN
 F 2 "Capacitor_SMD:C_0603_1608Metric_Pad1.05x0.95mm_HandSolder" H 5388 2350 50  0001 C CNN
@@
 AR Path="/5D0DF15B/5C6F0213" Ref="R59"  Part="1"
 AR Path="/5D1213F6/5C6F0213" Ref="R63"  Part="1"
-F 0 "R63" H 4770 3946 50  0000 L CNN
+F 0 "R37" H 4770 3946 50  0000 L CNN
 F 1 "22k" H 4770 3855 50  0000 L CNN
 F 2 "" V 4630 3900 50  0001 C CNN
@@
 AR Path="/5D0DF15B/5C6F0221" Ref="R57"  Part="1"
 AR Path="/5D1213F6/5C6F0221" Ref="R61"  Part="1"
-F 0 "R61" V 4243 3300 50  0000 C CNN
+F 0 "R35" V 4243 3300 50  0000 C CNN
 F 1 "10k" V 4334 3300 50  0000 C CNN
 F 2 "" V 4380 3300 50  0001 C CNN
@@
 AR Path="/5D0DF15B/5C6F0228" Ref="R56"  Part="1"
 AR Path="/5D1213F6/5C6F0228" Ref="R60"  Part="1"
-F 0 "R60" V 5143 2850 50  0000 C CNN
+F 0 "R34" V 5143 2850 50  0000 C CNN
 F 1 "22k" V 5234 2850 50  0000 C CNN
 F 2 "" V 5280 2850 50  0001 C CNN
@@
 AR Path="/5D0DF15B/5C6F0253" Ref="C62"  Part="1"
 AR Path="/5D1213F6/5C6F0253" Ref="C65"  Part="1"
-F 0 "C65" H 6115 2796 50  0000 L CNN
+F 0 "C52" H 6115 2796 50  0000 L CNN
 F 1 "100n 6V3 X5R" H 6115 2705 50  0000 L CNN
 F 2 "Capacitor_SMD:C_0603_1608Metric_Pad1.05x0.95mm_HandSolder" H 6038 2600 50  0001 C CNN
@@
 AR Path="/5D0DF15B/5C6F0260" Ref="C63"  Part="1"
 AR Path="/5D1213F6/5C6F0260" Ref="C66"  Part="1"
-F 0 "C66" H 6115 4546 50  0000 L CNN
+F 0 "C53" H 6115 4546 50  0000 L CNN
 F 1 "100n 6V3 X5R" H 6115 4455 50  0000 L CNN
 F 2 "Capacitor_SMD:C_0603_1608Metric_Pad1.05x0.95mm_HandSolder" H 6038 4350 50  0001 C CNN

Commit message: Schematic in progress.
Parts:
- R34, R35, R36, R37: footprint (none) -> Resistor_SMD:R_0603_1608Metric_Pad1.05x0.95mm_HandSolder
- U16: value LM6132A/NS -> TBD LM6132A/NS
Changed lines of the file:
@@
 AR Path="/5D0DF15B/5C6F01FE" Ref="U20"  Part="1"
 AR Path="/5D1213F6/5C6F01FE" Ref="U21"  Part="1"
-F 0 "U16" H 5500 3650 50  0000 L CNN
-F 1 "LM6132A/NS" H 5400 3350 50  0000 L CNN
+F 0 "U21" H 5500 3650 50  0000 L CNN
+F 1 "TBD LM6132A/NS" H 5400 3350 50  0000 L CNN
 F 2 "" H 5400 3550 50  0001 C CNN
 F 3 "http://www.analog.com/media/en/technical-documentation/data-sheets/AD8603_8607_8609.pdf" H 5400 3750 50  0001 C CNN
@@
 AR Path="/5D0DF15B/5C6F0205" Ref="R58"  Part="1"
 AR Path="/5D1213F6/5C6F0205" Ref="R62"  Part="1"
-F 0 "R36" V 4243 3650 50  0000 C CNN
+F 0 "R62" V 4243 3650 50  0000 C CNN
 F 1 "10k" V 4334 3650 50  0000 C CNN
-F 2 "" V 4380 3650 50  0001 C CNN
+F 2 "Resistor_SMD:R_0603_1608Metric_Pad1.05x0.95mm_HandSolder" V 4380 3650 50  0001 C CNN
 F 3 "~" H 4450 3650 50  0001 C CNN
 	1    4450 3650
@@
 AR Path="/5D0DF15B/5C6F020C" Ref="C61"  Part="1"
 AR Path="/5D1213F6/5C6F020C" Ref="C64"  Part="1"
-F 0 "C51" V 5098 2500 50  0000 C CNN
+F 0 "C64" V 5098 2500 50  0000 C CNN
 F 1 "1p" V 5189 2500 50  0000 C CNN
 F 2 "Capacitor_SMD:C_0603_1608Metric_Pad1.05x0.95mm_HandSolder" H 5388 2350 50  0001 C CNN
@@
 AR Path="/5D0DF15B/5C6F0213" Ref="R59"  Part="1"
 AR Path="/5D1213F6/5C6F0213" Ref="R63"  Part="1"
-F 0 "R37" H 4770 3946 50  0000 L CNN
+F 0 "R63" H 4770 3946 50  0000 L CNN
 F 1 "22k" H 4770 3855 50  0000 L CNN
-F 2 "" V 4630 3900 50  0001 C CNN
+F 2 "Resistor_SMD:R_0603_1608Metric_Pad1.05x0.95mm_HandSolder" V 4630 3900 50  0001 C CNN
 F 3 "~" H 4700 3900 50  0001 C CNN
 	1    4700 3900
@@
 AR Path="/5D0DF15B/5C6F0221" Ref="R57"  Part="1"
 AR Path="/5D1213F6/5C6F0221" Ref="R61"  Part="1"
-F 0 "R35" V 4243 3300 50  0000 C CNN
+F 0 "R61" V 4243 3300 50  0000 C CNN
 F 1 "10k" V 4334 3300 50  0000 C CNN
-F 2 "" V 4380 3300 50  0001 C CNN
+F 2 "Resistor_SMD:R_0603_1608Metric_Pad1.05x0.95mm_HandSolder" V 4380 3300 50  0001 C CNN
 F 3 "~" H 4450 3300 50  0001 C CNN
 	1    4450 3300
@@
 AR Path="/5D0DF15B/5C6F0228" Ref="R56"  Part="1"
 AR Path="/5D1213F6/5C6F0228" Ref="R60"  Part="1"
-F 0 "R34" V 5143 2850 50  0000 C CNN
+F 0 "R60" V 5143 2850 50  0000 C CNN
 F 1 "22k" V 5234 2850 50  0000 C CNN
-F 2 "" V 5280 2850 50  0001 C CNN
+F 2 "Resistor_SMD:R_0603_1608Metric_Pad1.05x0.95mm_HandSolder" V 5280 2850 50  0001 C CNN
 F 3 "~" H 5350 2850 50  0001 C CNN
 	1    5350 2850
@@
 AR Path="/5D0DF15B/5C6F0253" Ref="C62"  Part="1"
 AR Path="/5D1213F6/5C6F0253" Ref="C65"  Part="1"
-F 0 "C52" H 6115 2796 50  0000 L CNN
+F 0 "C65" H 6115 2796 50  0000 L CNN
 F 1 "100n 6V3 X5R" H 6115 2705 50  0000 L CNN
 F 2 "Capacitor_SMD:C_0603_1608Metric_Pad1.05x0.95mm_HandSolder" H 6038 2600 50  0001 C CNN
@@
 AR Path="/5D0DF15B/5C6F0260" Ref="C63"  Part="1"
 AR Path="/5D1213F6/5C6F0260" Ref="C66"  Part="1"
-F 0 "C53" H 6115 4546 50  0000 L CNN
+F 0 "C66" H 6115 4546 50  0000 L CNN
 F 1 "100n 6V3 X5R" H 6115 4455 50  0000 L CNN
 F 2 "Capacitor_SMD:C_0603_1608Metric_Pad1.05x0.95mm_HandSolder" H 6038 4350 50  0001 C CNN

Commit message: Schematic in progress.
Parts:
- U16: value TBD LM6132A/NS -> TBD
Changed lines of the file:
@@
 AR Path="/5D1213F6/5C6F01FE" Ref="U21"  Part="1"
 F 0 "U21" H 5500 3650 50  0000 L CNN
-F 1 "TBD LM6132A/NS" H 5400 3350 50  0000 L CNN
+F 1 "TBD" H 5400 3350 50  0000 L CNN
 F 2 "" H 5400 3550 50  0001 C CNN
 F 3 "http://www.analog.com/media/en/technical-documentation/data-sheets/AD8603_8607_8609.pdf" H 5400 3750 50  0001 C CNN
