File: uSensor_v1/uSensor_v1.sch (KiCad schematic (older format))
At the start: 130 parts

Commit message: Schematic in progress.
Parts:
- removed C? (x4): 100n 6V3 X5R, symbol Device:C
- removed C? (x4): 10n 6V3 X5R, symbol Device:C
- removed J?: KSS 213 Connector, symbol Connector_Generic_MountingPin:Conn_02x08_Odd_Even_MountingPin
- removed Q? (x2): Q_NPN_BCE, symbol Device:Q_NPN_BCE
- removed Q? (x2): Q_PNP_BCE, symbol Device:Q_PNP_BCE
- removed R? (x2): 10R, symbol Device:R
- removed R? (x6): 10k 1%, symbol Device:R
- removed R? (x2): 10k, symbol Device:R
- removed R? (x4): 1R, symbol Device:R
- removed U? (x2): LM6132A/NS, symbol Amplifier_Operational:AD8603
- added C? (x4): 10n 6V3 X5R, Capacitor_SMD:C_0603_1608Metric_Pad1.05x0.95mm_HandSolder, symbol Device:C
- added C? (x3): 100n 6V3 X5R, Capacitor_SMD:C_0603_1608Metric_Pad1.05x0.95mm_HandSolder, symbol Device:C
- added C?: 10u 6V3 X5R, Capacitor_SMD:C_0603_1608Metric_Pad1.05x0.95mm_HandSolder, symbol Device:C
- added C? (x2): 10u 6V3 Tantal, symbol Device:CP
- added U?: KSS-213, symbol Sentisa-IC:KSS-213
- added U?: AD5667, symbol Sentisa-IC:AD5667
- added U?: AD7795, symbol Sentisa-IC:AD7795
- C? (x6): footprint (none) -> Capacitor_SMD:C_0603_1608Metric_Pad1.05x0.95mm_HandSolder
- C?: value 100n -> 100n 6V3 X5R; footprint (none) -> Capacitor_SMD:C_0603_1608Metric_Pad1.05x0.95mm_HandSolder
- C?: value 10n -> 10n 6V3 X5R; footprint (none) -> Capacitor_SMD:C_0603_1608Metric_Pad1.05x0.95mm_HandSolder
- R?: value {R} -> TBD
Connections:
- net labels added: DAC_SCL, DAC_SDA, DAC_~CLR
- net labels removed: SENS_PDIC, SENS_VCC
- wire segments 552 -> 560
Other:
- note added: "COIL CURRENT SOURCES"
- note added: "Do ADC w procu,\nchyba że zostanie \nwolny kanał w \nzewnętrznym ADC"
- note added: "EXTERNAL ADC"
- note added: "EXTERNAL DAC"
- note added: "SENSORS SINGALS SUMMING CIRCUIT"
- note removed: "COIL CURRENT SOURCE - FOCUSING"
- note removed: "COIL CURRENT SOURCE - TRACKING"
- note removed: "Do ADC w procu, chyba że \nzostanie kanał w zewnętrznym ADC"
- note removed: "Podłączyć do zewnętrzengo DACA\n"
- moved on the sheet: C1, C?, J?, Q?, R1, R2, R3, R4, R5, R9, R?, RV?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

Commit message: Schematic in progress.
Parts:
- removed C?: 2u2 6v3 X5R, Capacitor_SMD:C_0603_1608Metric_Pad1.05x0.95mm_HandSolder, symbol Device:C
- removed C?: 2u2 6V3 X5R, Capacitor_SMD:C_0603_1608Metric_Pad1.05x0.95mm_HandSolder, symbol Device:C
- removed C? (x8): 100n 16V X5R, Capacitor_SMD:C_0603_1608Metric_Pad1.05x0.95mm_HandSolder, symbol Device:C
- removed C?: 1u 6V3 X5R, Capacitor_SMD:C_0603_1608Metric_Pad1.05x0.95mm_HandSolder, symbol Device:C
- removed D? (x2): LED, LED_SMD:LED_0603_1608Metric_Pad1.05x0.95mm_HandSolder, symbol Device:LED
- removed R?: 10k, Resistor_SMD:R_0603_1608Metric_Pad1.05x0.95mm_HandSolder, symbol Device:R
- removed R? (x2): 100R, Resistor_SMD:R_0603_1608Metric_Pad1.05x0.95mm_HandSolder, symbol Device:R
- removed U?: STM32F407VGTx, symbol MCU_ST_STM32F4:STM32F407VGTx
- added C?: 2u2 6v3 X5R, Capacitor_SMD:C_0603_1608Metric_Pad1.05x0.95mm_HandSolder, symbol Device:C
- added C?: 2u2 6V3 X5R, Capacitor_SMD:C_0603_1608Metric_Pad1.05x0.95mm_HandSolder, symbol Device:C
- added C? (x8): 100n 16V X5R, Capacitor_SMD:C_0603_1608Metric_Pad1.05x0.95mm_HandSolder, symbol Device:C
- added C?: 1u 6V3 X5R, Capacitor_SMD:C_0603_1608Metric_Pad1.05x0.95mm_HandSolder, symbol Device:C
- added C?: 22u 6V3 X5R, Capacitor_SMD:C_0603_1608Metric_Pad1.05x0.95mm_HandSolder, symbol Device:C
- added C?: 10u 6V3 X5R, Capacitor_SMD:C_0603_1608Metric_Pad1.05x0.95mm_HandSolder, symbol Device:C
- added D10, D7, D8, D9: TBD, Diode_THT:D_DO-201AE_P15.24mm_Horizontal, symbol Diode:1N62xxA
- added D? (x2): LED, LED_SMD:LED_0603_1608Metric_Pad1.05x0.95mm_HandSolder, symbol Device:LED
- added J5: USB_B_Mini, symbol Connector:USB_B_Mini
- added R24, R25: 22R, Resistor_SMD:R_0603_1608Metric_Pad1.05x0.95mm_HandSolder, symbol Device:R
- added R?: 10k, Resistor_SMD:R_0603_1608Metric_Pad1.05x0.95mm_HandSolder, symbol Device:R
- added R? (x2): 100R, Resistor_SMD:R_0603_1608Metric_Pad1.05x0.95mm_HandSolder, symbol Device:R
- added U?: STM32F407VGTx, Package_QFP:LQFP-100_14x14mm_P0.5mm, symbol Sentisa-Microcontrollers:STM32F407VGTx
- added U?: AZ1117-3.3, Package_TO_SOT_SMD:SOT-223-3_TabPin2, symbol Regulator_Linear:AZ1117-3.3
- gave numbers to parts that had none: 90
Connections:
- net labels added: USB_D+, USB_D-, USB_ID, USB_VBUS
- wire segments 560 -> 605
Other:
- note added: "PICKUP KSS-213"
- note added: "SWD CONNECTOR"
- note added: "USB CONNECTOR"
- note added: "VOLTAGE REGULATOR"
- note removed: "KSS 213"
- note removed: "Podłączyć do ADC procka"
- moved on the sheet: C1, C10, C11, C12, C14, C15, C19, C20, C21, C22, C23, C24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

Commit message: Schematic in progress.
Parts:
- removed C20: 100n 6V3 X5R, symbol Device:C
- removed R9: 6k, symbol Device:R
- removed U2, U3: LM6132A/NS, symbol Amplifier_Operational:AD8603
- added R13: 33R, symbol Device:R
- added U6: LM6132A, symbol Amplifier_Operational:LM358
- J2, J3: footprint (none) -> Connector_PinHeader_2.54mm:PinHeader_1x03_P2.54mm_Vertical
- R12: value 4k -> 33R
- R2: value 22k -> 220R
- R3: value 22k -> 10k
- RV1: value R_POT -> 10k
- gave numbers to parts that had none: 20
Connections:
- net +5V: now also U6.8 (V+)
- net DAC_SCL: now also U3.95 (TIM4_CH3/SDIO_D4/TIM10_CH1/DCMI_D6/ETH_MII_TXD3/I2C1_SCL/CAN1_RX/EVENTOUT/PB8)
- net DAC_SDA: now also U3.96 (SPI2_NSS/I2S2_WS/TIM4_CH4/TIM11_CH1/SDIO_D5/DCMI_D7/I2C1_SDA/CAN1_TX/EVENTOUT/PB9)
- net DAC_~CLR: now also U3.93 (I2C1_SDA/FSMC_NL/DCMI_VSYNC/USART1_RX/TIM4_CH2/EVENTOUT/PB7)
- net GND: now also U6.4 (V-); no longer R12.2
- net SENS_LD_PWR: now also R13.2; no longer Q1.3 (E)
- net TEMP_SENS_OUT_1: now also U3.15 (OTG_HS_ULPI_STP/EVENTOUT/ADC123_IN10/PC0)
- net TEMP_SENS_OUT_2: now also U3.16 (ETH_MDC/EVENTOUT/ADC123_IN11/PC1)
- net TEMP_SENS_OUT_3: now also U3.17 (SPI2_MISO/OTG_HS_ULPI_DIR/ETH_MII_TXD2/I2S2ext_SD/EVENTOUT/ADC123_IN12/PC2)
- net TEMP_SENS_OUT_4: now also U3.18 (SPI2_MOSI/I2S2_SD/OTG_HS_ULPI_NXT/ETH_MII_TX_CLK/EVENTOUT/ADC123_IN13/PC3)
- net at R3.1, R4.1: now also U6.1
- net at J3.3 (Pin_3), R5.1: now also U6.3 (+)
- net at R1.1, R2.1, R3.2: now also U6.2 (-)
- net at C1.1, Q2.1 (B): now also U6.7
- net at R12.1: now also Q2.3 (E)
- net at C1.2, R4.2: now also U6.6 (-)
- net at J2.3 (Pin_3): now also R12.2; no longer Q2.3 (E)
- net at RV1.2: now also U6.5 (+)
- net SENS_E: no longer names the net of U10.3 (E)
- net SENS_F: no longer names the net of U10.8 (F)
- net SENS_VR: no longer names the net of R19.1, U10.11 (VR)
- net VREF+: no longer names the net of U3.21 (VREF+)
- new net: Q1.3 (E), R13.1
- no-connect marks 3 -> 5
Other:
- note added: "DC/DC CONVERTER - OK"
- note added: "OLED DISPLAY - OK"
- note added: "PCB Temperature Sensors - OK"
- note added: "PWR FLAGS"
- note added: "SWD CONNECTOR - OK"
- note added: "TACT-SWITCH - OK"
- note added: "VOLTAGE REGULATOR - OK"
- note removed: "DC/DC CONVERTER"
- note removed: "Dodać sterowanie z DAC mikroprocka,\n wybor zworka na 3 goldpinach"
- note removed: "OLED DISPLAY"
- note removed: "PCB Temperature Sensors"
- note removed: "SWD CONNECTOR"
- note removed: "TACT-SWITCH"
- note removed: "VOLTAGE REGULATOR"
- note removed: "Złącze na PCB ma posiadać dokładne\noznaczenie polaryzacji"
- moved on the sheet: C1, C19, C31, C32, C33, C34, C38, C39, J2, J3, Q1, Q2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

Commit message: Schematic in progress.
Parts:
- R31: value 50R -> 51R
- U13, U14: value LM6132A/NS -> TBD
Connections:
- net +3V3: no longer C38.1, C39.1, U12.9 (VDD)
- net +5V: now also C38.1, C39.1, U12.9 (VDD)
- net REF_2.5V: now also U12.10 (Vref_IN)
- net ADC_SCLK: now reaches U11.1 (SCLK)
- net ADC_SCLK: now also U3.78 (SPI3_SCK/I2S3_CK/UART4_TX/SDIO_D2/DCMI_D8/USART3_TX/EVENTOUT/PC10)
- net ADC_DOUT: now reaches U11.23 (DOUT/~RDY)
- net ADC_DOUT: now also U3.79 (UART4_RX/SPI3_MISO/SDIO_D3/DCMI_D4/USART3_RX/I2S3ext_SD/EVENTOUT/PC11)
- net ADC_DIN: now reaches U11.24 (DIN)
- net ADC_DIN: now also U3.80 (UART5_TX/SDIO_CK/DCMI_D9/SPI3_MOSI/I2S3_SD/USART3_CK/EVENTOUT/PC12)
- net ADC_~CS: now reaches U11.3 (~CS)
- net ADC_~CS: now also U3.66 (I2S_CKIN/MCO2/TIM8_CH4/SDIO_D1/I2C3_SDA/DCMI_D3/TIM3_CH4/EVENTOUT/PC9)
Other:
- note added: "Czy dajemy \nkompensację weściowego \nnapęcia niezrównoważenia?"
- note added: "Jaka to wersja układu?\nZ referencją czy bez?"
- note added: "Jaki zakres sygnału \nwyjściowego?"
- moved on the sheet: C19
Changed lines of the file:
@@
 L Device:C C19
 U 1 1 5C094316
-P 4500 24550
-F 0 "C19" H 4615 24596 50  0000 L CNN
-F 1 "100n 6V3 X5R" H 4615 24505 50  0000 L CNN
-F 2 "" H 4538 24400 50  0001 C CNN
-F 3 "~" H 4500 24550 50  0001 C CNN
-	1    4500 24550
+P 4500 24400
+F 0 "C19" H 4615 24446 50  0000 L CNN
+F 1 "100n 6V3 X5R" H 4615 24355 50  0000 L CNN
+F 2 "" H 4538 24250 50  0001 C CNN
+F 3 "~" H 4500 24400 50  0001 C CNN
+	1    4500 24400
 	1    0    0    -1
 $EndComp
@@
 $EndComp
 Wire Wire Line
-	4500 24700 4500 24800
+	4500 24550 4500 24800
 $Comp
 L Device:C C1
@@
 P 6550 18200
 F 0 "U13" H 6550 18350 50  0000 L CNN
-F 1 "LM6132A/NS" H 6550 18050 50  0000 L CNN
+F 1 "TBD" H 6550 18050 50  0000 L CNN
 F 2 "" H 6550 18200 50  0001 C CNN
 F 3 "http://www.analog.com/media/en/technical-documentation/data-sheets/AD8603_8607_8609.pdf" H 6550 18400 50  0001 C CNN
@@
 P 8300 18300
 F 0 "U14" H 8450 18400 50  0000 L CNN
-F 1 "LM6132A/NS" H 8450 18200 50  0000 L CNN
+F 1 "TBD" H 8450 18200 50  0000 L CNN
 F 2 "" H 8300 18300 50  0001 C CNN
 F 3 "http://www.analog.com/media/en/technical-documentation/data-sheets/AD8603_8607_8609.pdf" H 8300 18500 50  0001 C CNN
@@
 P 9250 18300
 F 0 "R31" V 9457 18300 50  0000 C CNN
-F 1 "50R" V 9366 18300 50  0000 C CNN
+F 1 "51R" V 9366 18300 50  0000 C CNN
 F 2 "" V 9180 18300 50  0001 C CNN
 F 3 "~" H 9250 18300 50  0001 C CNN
@@
 L power:+3V3 #PWR026
 U 1 1 624965A6
-P 6300 13500
-F 0 "#PWR026" H 6300 13350 50  0001 C CNN
-F 1 "+3V3" H 6315 13673 50  0000 C CNN
-F 2 "" H 6300 13500 50  0001 C CNN
-F 3 "" H 6300 13500 50  0001 C CNN
-	1    6300 13500
+P 6100 13500
+F 0 "#PWR026" H 6100 13350 50  0001 C CNN
+F 1 "+3V3" H 6115 13673 50  0000 C CNN
+F 2 "" H 6100 13500 50  0001 C CNN
+F 3 "" H 6100 13500 50  0001 C CNN
+	1    6100 13500
 	1    0    0    -1
 $EndComp
-Text Notes 6450 13500 0    150  ~ 30
+Text Notes 6400 13450 0    150  ~ 30
 ?
 Wire Wire Line
@@
 	3900 24000 3900 23900
 Wire Wire Line
-	4500 24000 4500 24400
+	4500 24000 4500 24250
 Wire Wire Line
 	3900 24100 3900 24000
@@
 Wire Wire Line
 	12600 4400 14200 4400
-Text GLabel 11000 9850 2    40   Input ~ 0
+Text GLabel 11150 9850 2    40   Input ~ 0
 TEMP_SENS_OUT_1
-Text GLabel 11000 9950 2    40   Input ~ 0
+Text GLabel 11150 9950 2    40   Input ~ 0
 TEMP_SENS_OUT_2
-Text GLabel 11000 10050 2    40   Input ~ 0
+Text GLabel 11150 10050 2    40   Input ~ 0
 TEMP_SENS_OUT_3
-Text GLabel 11000 10150 2    40   Input ~ 0
+Text GLabel 11150 10150 2    40   Input ~ 0
 TEMP_SENS_OUT_4
 Wire Wire Line
-	10400 9850 11000 9850
+	10400 9850 11150 9850
 Wire Wire Line
-	11000 9950 10400 9950
+	11150 9950 10400 9950
 Wire Wire Line
-	10400 10050 11000 10050
+	10400 10050 11150 10050
 Wire Wire Line
-	11000 10150 10400 10150
+	11150 10150 10400 10150
 $Comp
 L power:+5V #PWR0106
@@
 Wire Wire Line
 	11250 8850 10400 8850
-Text GLabel 14300 15550 2    50   Input ~ 0
-FOC_ERR_2_ADC
+Text Notes 9350 18600 0    50   ~ 0
+Jaki zakres sygnału \nwyjściowego?
+Wire Notes Line
+	9100 17900 9100 18850
+Wire Notes Line
+	9100 18850 10300 18850
+Wire Notes Line
+	10300 18850 10300 17900
+Wire Notes Line
+	10300 17900 9100 17900
+Wire Notes Line
+	5300 16600 6650 16600
+Wire Notes Line
+	6650 16600 6650 17300
+Wire Notes Line
+	6650 17300 5300 17300
+Wire Notes Line
+	5300 17300 5300 16600
+Text Notes 5450 17100 0    50   ~ 0
+Czy dajemy \nkompensację weściowego \nnapęcia niezrównoważenia?
+$Comp
+L power:+5V #PWR0107
+U 1 1 69068D29
+P 6300 13500
+F 0 "#PWR0107" H 6300 13350 50  0001 C CNN
+F 1 "+5V" H 6315 13673 50  0000 C CNN
+F 2 "" H 6300 13500 50  0001 C CNN
+F 3 "" H 6300 13500 50  0001 C CNN
+	1    6300 13500
+	1    0    0    -1
+$EndComp
+Wire Notes Line
+	7600 14150 8550 14150
+Wire Notes Line
+	8550 14150 8550 14650
+Wire Notes Line
+	8550 14650 7600 14650
+Wire Notes Line
+	7600 14650 7600 14150
+Text Notes 7600 14350 0    50   ~ 0
+Jaka to wersja układu?\nZ referencją czy bez?
+Text GLabel 6450 14650 0    50   Input ~ 0
+REF_2.5V
+Wire Wire Line
+	6450 14650 6550 14650
+Wire Notes Line
+	5850 14400 6550 14400
+Wire Notes Line
+	6550 14400 6550 14750
+Wire Notes Line
+	6550 14750 5850 14750
+Wire Notes Line
+	5850 14750 5850 14400
+Text Notes 5900 14700 0    150  ~ 30
+?
+Wire Notes Line
+	15250 4100 15250 4550
+Wire Notes Line
+	15250 4550 14250 4550
+Wire Notes Line
+	14250 4550 14250 4100
+Wire Notes Line
+	14250 4100 15250 4100
+Text Notes 15000 4450 0    150  ~ 30
+?
+$Comp
+L power:GNDA #PWR0110
+U 1 1 694403F9
+P 5550 28400
+F 0 "#PWR0110" H 5550 28150 50  0001 C CNN
+F 1 "GNDA" H 5555 28227 50  0000 C CNN
+F 2 "" H 5550 28400 50  0001 C CNN
+F 3 "" H 5550 28400 50  0001 C CNN
+	1    5550 28400
+	1    0    0    -1
+$EndComp
+$Comp
+L power:GNDD #PWR0111
+U 1 1 69440627
+P 5950 28400
+F 0 "#PWR0111" H 5950 28150 50  0001 C CNN
+F 1 "GNDD" H 5954 28245 50  0000 C CNN
+F 2 "" H 5950 28400 50  0001 C CNN
+F 3 "" H 5950 28400 50  0001 C CNN
+	1    5950 28400
+	1    0    0    -1
+$EndComp
+$Comp
+L power:PWR_FLAG #FLG0104
+U 1 1 6944091F
+P 5550 28300
+F 0 "#FLG0104" H 5550 28375 50  0001 C CNN
+F 1 "PWR_FLAG" H 5550 28474 50  0000 C CNN
+F 2 "" H 5550 28300 50  0001 C CNN
+F 3 "~" H 5550 28300 50  0001 C CNN
+	1    5550 28300
+	1    0    0    -1
+$EndComp
+Wire Wire Line
+	5550 28300 5550 28400
+$Comp
+L power:PWR_FLAG #FLG0105
+U 1 1 69519361
+P 5950 28300
+F 0 "#FLG0105" H 5950 28375 50  0001 C CNN
+F 1 "PWR_FLAG" H 5950 28474 50  0000 C CNN
+F 2 "" H 5950 28300 50  0001 C CNN
+F 3 "~" H 5950 28300 50  0001 C CNN
+	1    5950 28300
+	1    0    0    -1
+$EndComp
+Wire Wire Line
+	5950 28300 5950 28400
+Text GLabel 11450 17300 0    40   Input ~ 0
+ADC_~CS
+Wire Wire Line
+	11450 17300 11550 17300
+Text GLabel 14050 14800 2    40   Output ~ 0
+ADC_DOUT
+Text GLabel 14050 14900 2    40   Input ~ 0
+ADC_DIN
+Text GLabel 14050 15000 2    40   BiDi ~ 0
+ADC_SCLK
+Wire Wire Line
+	14050 14800 13950 14800
+Wire Wire Line
+	13950 14900 14050 14900
+Wire Wire Line
+	14050 15000 13950 15000
+Text GLabel 11150 10950 2    40   Input ~ 0
+ADC_DOUT
+Text GLabel 11150 11050 2    40   Output ~ 0
+ADC_DIN
+Text GLabel 11150 10850 2    40   BiDi ~ 0
+ADC_SCLK
+Text GLabel 11150 10750 2    40   Output ~ 0
+ADC_~CS
+Wire Wire Line
+	11150 11050 10400 11050
+Wire Wire Line
+	11150 10950 10400 10950
+Wire Wire Line
+	11150 10850 10400 10850
+Wire Wire Line
+	11150 10750 10400 10750
+Wire Notes Line
+	5800 15050 6700 15050
+Wire Notes Line
+	6700 15050 6700 15300
+Wire Notes Line
+	6700 15300 5800 15300
+Wire Notes Line
+	5800 15300 5800 15050
+Text Notes 5850 15300 0    150  ~ 30
+?
 $EndSCHEMATC

Commit message: Schematic in progress.
Parts:
- removed D10, D7: TBD, Diode_THT:D_DO-201AE_P15.24mm_Horizontal, symbol Diode:1N62xxA
Connections:
- net USB_D+: no longer U3.71 (USART1_RTS/CAN1_TX/TIM1_ETR/OTG_FS_DP/EVENTOUT/PA12)
- net USB_D-: no longer U3.70 (USART1_CTS/CAN1_RX/TIM1_CH4_/OTG_FS_DM/EVENTOUT/PA11)
- net USB_ID: no longer J5.4 (ID), U3.69 (USART1_RX/TIM1_CH3/OTG_FS_ID/DCMI_D1/EVENTOUT/PA10)
- net USB_VBUS: no longer J5.1 (VBUS), U3.68 (USART1_TX/TIM1_CH2/I2C3_SMBA/DCMI_D0/EVENTOUT/OTG_FS_VBUS/PA9)
- no-connect marks 5 -> 7
Other:
- note added: "USB CONNECTOR-NOK"
- note removed: "USB CONNECTOR"
Changed lines of the file:
@@
 Wire Wire Line
 	6050 17600 6300 17600
-Text Notes 5400 18300 0    50   ~ 0
+Text Notes 5450 18300 0    50   ~ 0
 A
-Text Notes 5400 17800 0    50   ~ 0
+Text Notes 5450 17800 0    50   ~ 0
 B
-Text Notes 5400 18600 0    50   ~ 0
+Text Notes 5450 18600 0    50   ~ 0
 C
-Text Notes 5400 18100 0    50   ~ 0
+Text Notes 5450 18100 0    50   ~ 0
 D
 Wire Wire Line
@@
 Wire Wire Line
 	13200 4650 13900 4650
-Text GLabel 14400 5050 2    50   BiDi ~ 0
-USB_ID
-Wire Wire Line
-	14400 5050 13300 5050
-$Comp
-L Diode:1N62xxA D10
-U 1 1 636216C0
-P 14200 5300
-F 0 "D10" V 14154 5379 50  0000 L CNN
-F 1 "TBD" V 14245 5379 50  0000 L CNN
-F 2 "Diode_THT:D_DO-201AE_P15.24mm_Horizontal" H 14200 5100 50  0001 C CNN
-F 3 "https://www.vishay.com/docs/88301/15ke.pdf" H 14150 5300 50  0001 C CNN
-	1    14200 5300
-	0    1    1    0
-$EndComp
 $Comp
 L Diode:1N62xxA D9
@@
 	0    1    1    0
 $EndComp
-$Comp
-L Diode:1N62xxA D7
-U 1 1 636210BD
-P 13300 5300
-F 0 "D7" V 13254 5379 50  0000 L CNN
-F 1 "TBD" V 13345 5379 50  0000 L CNN
-F 2 "Diode_THT:D_DO-201AE_P15.24mm_Horizontal" H 13300 5100 50  0001 C CNN
-F 3 "https://www.vishay.com/docs/88301/15ke.pdf" H 13250 5300 50  0001 C CNN
-	1    13300 5300
-	0    1    1    0
-$EndComp
-Wire Wire Line
-	13300 5150 13300 5050
-Connection ~ 13300 5050
-Wire Wire Line
-	13300 5050 12600 5050
 Wire Wire Line
 	13600 5150 13600 4950
@@
 Wire Wire Line
 	13900 4650 14400 4650
-Wire Wire Line
-	12600 4650 12600 4400
-Wire Wire Line
-	14200 4400 14400 4400
 $Comp
 L power:GND #PWR033
@@
 	13300 5550 13600 5550
 Wire Wire Line
-	14200 5550 14200 5450
-Connection ~ 13300 5550
-Wire Wire Line
-	13300 5550 13300 5450
-Wire Wire Line
 	13900 5450 13900 5550
-Connection ~ 13900 5550
-Wire Wire Line
-	13900 5550 14200 5550
 Wire Wire Line
 	13600 5450 13600 5550
@@
 Wire Wire Line
 	13600 5550 13900 5550
-Text GLabel 14400 4400 2    50   BiDi ~ 0
-USB_VBUS
 Text Notes 11950 4150 0    150  ~ 30
-USB CONNECTOR
+USB CONNECTOR-NOK
 Wire Notes Line
 	11950 3900 15400 3900
@@
 Wire Wire Line
 	11100 6450 10400 6450
-Text GLabel 10500 7650 2    50   BiDi ~ 0
+Text GLabel 11100 7650 2    50   BiDi ~ 0
 USB_D+
-Text GLabel 10500 7550 2    50   BiDi ~ 0
+Text GLabel 11100 7550 2    50   BiDi ~ 0
 USB_D-
-Text GLabel 10500 7450 2    50   BiDi ~ 0
-USB_ID
-Text GLabel 11100 7350 2    50   BiDi ~ 0
-USB_VBUS
-Wire Wire Line
-	11100 7350 10400 7350
-Wire Wire Line
-	10500 7450 10400 7450
-Wire Wire Line
-	10400 7550 10500 7550
-Wire Wire Line
-	10500 7650 10400 7650
 $Comp
 L Sentisa-Microcontrollers:STM32F407VGTx U3
@@
 Wire Wire Line
 	4750 29150 4750 29050
-Wire Wire Line
-	14200 5150 14200 4400
-Connection ~ 14200 4400
-Wire Wire Line
-	12600 4400 14200 4400
 Text GLabel 11150 9850 2    40   Input ~ 0
 TEMP_SENS_OUT_1
@@
 Text Notes 5900 14700 0    150  ~ 30
 ?
-Wire Notes Line
-	15250 4100 15250 4550
-Wire Notes Line
-	15250 4550 14250 4550
-Wire Notes Line
-	14250 4550 14250 4100
-Wire Notes Line
-	14250 4100 15250 4100
-Text Notes 15000 4450 0    150  ~ 30
-?
 $Comp
 L power:GNDA #PWR0110
@@
 	11150 10750 10400 10750
 Wire Notes Line
-	5800 15050 6700 15050
+	6250 15000 6700 15000
 Wire Notes Line
-	6700 15050 6700 15300
+	6700 15000 6700 15250
 Wire Notes Line
-	6700 15300 5800 15300
+	6700 15250 6250 15250
 Wire Notes Line
-	5800 15300 5800 15050
-Text Notes 5850 15300 0    150  ~ 30
+	6250 15250 6250 15000
+Text Notes 6350 15250 0    150  ~ 30
 ?
+NoConn ~ 12600 4650
+NoConn ~ 12600 5050
+Text GLabel 11100 7450 2    50   BiDi ~ 0
+USB_ID
+Text GLabel 11100 7350 2    50   BiDi ~ 0
+USB_VBUS
+Text GLabel 14300 4400 2    50   BiDi ~ 0
+USB_VBUS
+Text GLabel 14300 4500 2    50   BiDi ~ 0
+USB_ID
 $EndSCHEMATC

Commit message: Schematic in progress.
Parts:
- removed D8, D9: TBD, Diode_THT:D_DO-201AE_P15.24mm_Horizontal, symbol Diode:1N62xxA
- removed J5: USB_B_Mini, symbol Connector:USB_B_Mini
- added J5: USB_B, Connector_USB:USB_B_OST_USB-B1HSxx_Horizontal, symbol Sentisa-Connectors:USB_B
- added U22: RCLAMP, symbol Sentisa-IC:RCLAMP
- C1, C19: footprint (none) -> Capacitor_SMD:C_0603_1608Metric_Pad1.05x0.95mm_HandSolder
- C21, C22, C23, C24: value 100n -> 100n 6V3 X5R; footprint (none) -> Capacitor_SMD:C_0603_1608Metric_Pad1.05x0.95mm_HandSolder
- C31, C34: footprint (none) -> Capacitor_Tantalum_SMD:CP_EIA-3216-10_Kemet-I_Pad1.58x1.35mm_HandSolder
- L1, L3: footprint (none) -> Sentisa-Coils:FERROCORE_DLG-1005-101; MPN DE1205-100 -> DLG-1005-101
- L2: footprint (none) -> Sentisa-Coils:FERROCORE_DLG-0705-120
- Q1, Q2, R12, R13, R19: footprint (none) -> TBD
- R1, R11, R2, R26, R27, R28, R29, R3, R30, R31, R32, R33, R4, R5, R8: footprint (none) -> Resistor_SMD:R_0603_1608Metric_Pad1.05x0.95mm_HandSolder
- RV1: footprint (none) -> Sentisa-Resistors:Potentiometer_SR_Passives_T910W_Vertical; MFR (none) -> SR Passives; MPN (none) -> T910W-10K
- SW1, SW2: footprint (none) -> Button_Switch_THT:SW_PUSH_6mm_H4.3mm; MFR (none) -> Ninigi; MPN (none) -> TACT-67N-F
- U1: footprint (none) -> Sentisa-IC:AIMTEC_AM10TW-2405DZ
- U6: footprint (none) -> Sentisa-IC:SO-8
Connections:
- net +5V: now also U22.5 (VCC)
- net FOC_ERR_2_ADC: now also U11.7 (AIN1(+))
- net GND: now also J5.4 (GND), J5.5 (Shield), U22.2 (GND)
- net USB_D+: now also U3.71 (USART1_RTS/CAN1_TX/TIM1_ETR/OTG_FS_DP/EVENTOUT/PA12), U22.3 (D2)
- net USB_D-: now also U3.70 (USART1_CTS/CAN1_RX/TIM1_CH4_/OTG_FS_DM/EVENTOUT/PA11), U22.1 (D1)
- net USB_VBUS: now also U3.68 (USART1_TX/TIM1_CH2/I2C3_SMBA/DCMI_D0/EVENTOUT/OTG_FS_VBUS/PA9), J5.1 (VBUS), U22.4 (D3)
- net at R25.2: now also J5.2 (D-)
- net at R24.2: now also J5.3 (D+)
- net SWCLK renamed PROG_SWCLK
- net SWDIO renamed PROG_SWDIO
- net SWO renamed PROG_SWO
- net ~RST renamed PROG_~RST
- no-connect marks 7 -> 77
Other:
- note added: "FT"
- note added: "USB CONNECTOR-OK"
- note removed: "USB CONNECTOR-NOK"
- moved on the sheet: C19, C21, C22, C23, C24, C31, C32, C33, C34, R24, R25, U11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
