File: uSensor_v1/uSensor_v1.sch (KiCad schematic (older format))
At the start: 119 parts, among them J1 +12V Supply, J2 Conn_01x03, J3 Conn_01x03, J4 NS25-W8P 6-pin 2,54mm, J5 USB_B, Q1 BC817-25T116, Q2 BC817-25T116, SW1 SW_Push, SW2 SW_Push, U1 AM10TW-2405DZ, U10 KSS-213, U11 AD7795, U12 AD5667, U13 TBD, U14 TBD, U15 REF192, U2 AZ1117-3.3, U22 RCLAMP, U3 STM32F407VGTx, U4 MCP9700AT, U5 MCP9700AT, U6 LM6132A, U7 MCP9700AT, U8 MCP9700AT, U9 UG-2864KSWLG01

Commit message: Schematic in progress.
Parts:
- U10, U12, U9: footprint (none) -> TBD
- U11: footprint (none) -> Sentisa-IC:TSSOP-24_4.4x7.8mm_Pitch0.65mm
- U15: footprint (none) -> Sentisa-IC:SO-8; MFR (none) -> Analog Devices; MPN (none) -> REF192FSZ
- U22: footprint (none) -> Sentisa-IC:SOT-23-6
Connections:
- net FOC_ERR_2_ADC: no longer U11.7 (AIN1(+))
- no-connect marks 77 -> 61
Other:
- note added: "DC/DC CONVERTER"
- note added: "OLED DISPLAY"
- note added: "PCB Temperature Sensors"
- note added: "SWD CONNECTOR"
- note added: "TACT-SWITCH"
- note added: "USB CONNECTOR"
- note added: "VOLTAGE REGULATOR"
- note removed: "DC/DC CONVERTER - OK"
- note removed: "OLED DISPLAY - OK"
- note removed: "PCB Temperature Sensors - OK"
- note removed: "SWD CONNECTOR - OK"
- note removed: "TACT-SWITCH - OK"
- note removed: "USB CONNECTOR-OK"
- note removed: "VOLTAGE REGULATOR - OK"
Changed lines of the file:
@@
 	19650 7100 19950 7100
 Text Notes 17950 4150 0    150  ~ 30
-OLED DISPLAY - OK
+OLED DISPLAY
 Wire Notes Line
 	17900 3900 22600 3900
@@
 F 0 "U9" H 19400 7650 50  0000 C CNN
 F 1 "UG-2864KSWLG01" H 18800 7650 50  0000 C CNN
-F 2 "" H 19050 6050 50  0001 C CNN
+F 2 "TBD" H 19050 6050 50  0001 C CNN
 F 3 "" H 19050 6050 50  0001 C CNN
 F 4 "WiseChip" H 18950 6050 50  0001 C CNN "MFR"
@@
 	16200 6900 16300 6900
 Text Notes 15550 4150 0    150  ~ 30
-TACT-SWITCH - OK
+TACT-SWITCH
 Wire Notes Line
 	15500 3900 15500 8000
@@
 	1150 14800 1150 14700
 Text Notes 11950 8350 0    150  ~ 30
-PCB Temperature Sensors - OK
+PCB Temperature Sensors
 $Comp
 L Sensor_Temperature:MCP9700AT-ETT U4
@@
 F 0 "U15" H 1100 21000 50  0000 L CNN
 F 1 "REF192" H 1450 21000 50  0000 L CNN
-F 2 "" H 1400 20700 50  0001 C CIN
+F 2 "Sentisa-IC:SO-8" H 1400 20700 50  0001 C CIN
 F 3 "http://www.analog.com/static/imported-files/data_sheets/REF19xSeries.pdf" H 1400 20700 50  0001 C CIN
+F 4 "Analog Devices" H 1400 20750 50  0001 C CNN "MFR"
+F 5 "REF192FSZ" H 1400 20750 50  0001 C CNN "MPN"
 	1    1400 20750
 	1    0    0    -1
@@
 $EndComp
 Text Notes 600  800  0    150  ~ 30
-DC/DC CONVERTER - OK
+DC/DC CONVERTER
 $Comp
 L Sentisa-IC:AM10TW-2405DZ U1
@@
 F 0 "U10" H 3200 15650 50  0000 C CNN
 F 1 "KSS-213" H 3950 15650 50  0000 C CNN
-F 2 "" H 3650 15000 50  0001 C CNN
+F 2 "TBD" H 3650 15000 50  0001 C CNN
 F 3 "file:///C:/Users/Micha%C5%82/Desktop/Temp_Files/sony_1944121.pdf" H 3650 15000 50  0001 C CNN
 	1    3650 15000
@@
 F 0 "U12" H 6800 15700 50  0000 C CNN
 F 1 "AD5667" H 7800 15700 50  0000 C CNN
-F 2 "" H 7350 15050 50  0001 C CNN
+F 2 "TBD" H 7350 15050 50  0001 C CNN
 F 3 "https://www.tme.eu/pl/Document/3f74630f87cd4a86155519503328f287/AD5667BRMZ-Analog-Devices.pdf" H 7350 15050 50  0001 C CNN
 F 4 "Analog Devices" H 7350 15100 50  0001 C CNN "MFR"
@@
 F 0 "U11" H 13050 17450 50  0000 C CNN
 F 1 "AD7795" H 14850 17450 50  0000 C CNN
-F 2 "" H 14000 16350 50  0001 C CNN
+F 2 "Sentisa-IC:TSSOP-24_4.4x7.8mm_Pitch0.65mm" H 14000 16350 50  0001 C CNN
 F 3 "https://www.tme.eu/pl/Document/a63c7cd0d240f04c7b735f80a1ec0e97/AD7794_7795.pdf" H 14000 16350 50  0001 C CNN
 F 4 "Analog Devices" H 14000 16050 50  0001 C CNN "MFR"
@@
 USB_D-
 Text Notes 11950 3450 0    150  ~ 30
-USB CONNECTOR-OK
+USB CONNECTOR
 Text Notes 11950 6400 0    150  ~ 30
-SWD CONNECTOR - OK
+SWD CONNECTOR
 Wire Notes Line
 	11950 6150 15400 6150
@@
 	550  3900 11850 3900
 Text Notes 8000 800  0    150  ~ 30
-VOLTAGE REGULATOR - OK
+VOLTAGE REGULATOR
 $Comp
 L Regulator_Linear:AZ1117-3.3 U2
@@
 F 0 "U22" H 13750 5600 50  0000 L CNN
 F 1 "RCLAMP" H 14100 5600 50  0000 L CNN
-F 2 "" H 14050 5300 50  0001 C CNN
+F 2 "Sentisa-IC:SOT-23-6" H 14050 5300 50  0001 C CNN
 F 3 "https://www.tme.eu/pl/Document/f3858518c628a8bfddce32a44cc019aa/RCLAMP0504S.pdf" H 14050 5300 50  0001 C CNN
 F 4 "Semtech" H 14050 5300 50  0001 C CNN "MFR"
@@
 Wire Wire Line
 	12200 4650 12200 4750
-NoConn ~ 12800 14800
-NoConn ~ 12800 14900
-NoConn ~ 12800 15200
-NoConn ~ 12800 15400
-NoConn ~ 12800 15500
-NoConn ~ 12800 15700
-NoConn ~ 12800 15800
-NoConn ~ 12800 16000
-NoConn ~ 12800 16100
-NoConn ~ 12800 16300
-NoConn ~ 12800 16400
-NoConn ~ 12800 16600
-NoConn ~ 12800 16700
-NoConn ~ 12800 16900
-NoConn ~ 12800 17100
-NoConn ~ 6550 15150
 Text GLabel 9500 18300 2    50   Output ~ 0
 FOC_ERR_2_ADC
@@
 Wire Wire Line
 	5650 29050 5650 29150
-Wire Wire Line
-	11750 15100 12800 15100
 $Comp
 L power:GND #PWR0118
@@
 	1    0    0    -1
 $EndComp
+Wire Wire Line
+	12450 14900 12450 15200
+Connection ~ 12450 15200
+Text GLabel 11750 14800 0    50   Input ~ 0
+REF_2.5V
+Wire Wire Line
+	11750 14800 12550 14800
+Wire Wire Line
+	12450 14900 12550 14900
+Wire Wire Line
+	12550 15100 11750 15100
 $EndSCHEMATC

Commit message: Schematic in progress.
Parts:
- added R? (x2): 22k, Resistor_SMD:R_0603_1608Metric_Pad1.05x0.95mm_HandSolder, symbol Device:R
- added RV?: 10k, Sentisa-Resistors:Potentiometer_SR_Passives_T910W_Vertical, symbol Device:R_POT
Connections:
- net +3V3: now also C38.1, C39.1, U12.9 (VDD)
- net +5V: now also R?.2; no longer C38.1, C39.1, U12.9 (VDD)
- net -5V: now also R?.2
- net at R26.1, R30.1, R32.1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: now also RV?.2
- new net: R?.1, RV?.1
- new net: R?.1, RV?.3
Other:
- note added: "!"
- note added: "LOGIC INPUTS (ADDR, ~CLR~, ~LDAC~):\nV_INL = 0.15xVDD MAX\nV_INH = 0.85xVDD MIN\n\nLOGIC INPUTS (SDA, SCL):\nV_INL = 0.3xVDD MAX\nV_INH = 0.7xVDD MIN"
- note removed: "Czy dajemy \nkompensację weściowego \nnapęcia niezrównoważenia?"
Changed lines of the file:
@@
 L power:+3V3 #PWR026
 U 1 1 624965A6
-P 6100 13500
-F 0 "#PWR026" H 6100 13350 50  0001 C CNN
-F 1 "+3V3" H 6115 13673 50  0000 C CNN
-F 2 "" H 6100 13500 50  0001 C CNN
-F 3 "" H 6100 13500 50  0001 C CNN
-	1    6100 13500
+P 6300 13500
+F 0 "#PWR026" H 6300 13350 50  0001 C CNN
+F 1 "+3V3" H 6315 13673 50  0000 C CNN
+F 2 "" H 6300 13500 50  0001 C CNN
+F 3 "" H 6300 13500 50  0001 C CNN
+	1    6300 13500
 	1    0    0    -1
 $EndComp
@@
 	14100 13600 14100 14500
 Wire Notes Line
-	10650 12800 16050 12800
-Wire Notes Line
-	16050 12800 16050 18050
-Wire Notes Line
-	16050 18050 10650 18050
+	10650 12800 16800 12800
+Wire Notes Line
+	16800 12800 16800 18050
+Wire Notes Line
+	16800 18050 10650 18050
 Wire Notes Line
 	10650 18050 10650 12800
@@
 Wire Notes Line
 	10300 17900 9100 17900
-Wire Notes Line
-	5300 16600 6650 16600
-Wire Notes Line
-	6650 16600 6650 17300
-Wire Notes Line
-	6650 17300 5300 17300
-Wire Notes Line
-	5300 17300 5300 16600
-Text Notes 5450 17100 0    50   ~ 0
-Czy dajemy \nkompensację weściowego \nnapęcia niezrównoważenia?
 $Comp
 L power:+5V #PWR0107
 U 1 1 69068D29
-P 6300 13500
-F 0 "#PWR0107" H 6300 13350 50  0001 C CNN
-F 1 "+5V" H 6315 13673 50  0000 C CNN
-F 2 "" H 6300 13500 50  0001 C CNN
-F 3 "" H 6300 13500 50  0001 C CNN
-	1    6300 13500
+P 6100 13500
+F 0 "#PWR0107" H 6100 13350 50  0001 C CNN
+F 1 "+5V" H 6115 13673 50  0000 C CNN
+F 2 "" H 6100 13500 50  0001 C CNN
+F 3 "" H 6100 13500 50  0001 C CNN
+	1    6100 13500
 	1    0    0    -1
 $EndComp
@@
 Wire Wire Line
 	12550 15100 11750 15100
+Text Notes 10400 8850 0    50   ~ 0
+FT
+Text Notes 10400 8950 0    50   ~ 0
+FT
+Text Notes 10400 9050 0    50   ~ 0
+FT
+Text Notes 8300 15500 0    50   ~ 0
+LOGIC INPUTS (ADDR, ~CLR~, ~LDAC~):\nV_INL = 0.15xVDD MAX\nV_INH = 0.85xVDD MIN\n\nLOGIC INPUTS (SDA, SCL):\nV_INL = 0.3xVDD MAX\nV_INH = 0.7xVDD MIN
+Wire Notes Line
+	9650 14900 9650 15550
+Wire Notes Line
+	9650 15550 8250 15550
+Wire Notes Line
+	8250 15550 8250 14900
+Wire Notes Line
+	8250 14900 9650 14900
+Text Notes 9350 15350 0    150  ~ 30
+!
+$Comp
+L Device:R_POT RV?
+U 1 1 5C5A9E6C
+P 6050 17250
+F 0 "RV?" V 5843 17250 50  0000 C CNN
+F 1 "10k" V 5934 17250 50  0000 C CNN
+F 2 "Sentisa-Resistors:Potentiometer_SR_Passives_T910W_Vertical" H 6050 17250 50  0001 C CNN
+F 3 "~" H 6050 17250 50  0001 C CNN
+F 4 "SR Passives" H 6050 17250 50  0001 C CNN "MFR"
+F 5 "T910W-10K" H 6050 17250 50  0001 C CNN "MPN"
+	1    6050 17250
+	0    1    1    0
+$EndComp
+$Comp
+L Device:R R?
+U 1 1 5C5AB220
+P 6300 17000
+F 0 "R?" H 6230 16954 50  0000 R CNN
+F 1 "22k" H 6230 17045 50  0000 R CNN
+F 2 "Resistor_SMD:R_0603_1608Metric_Pad1.05x0.95mm_HandSolder" V 6230 17000 50  0001 C CNN
+F 3 "~" H 6300 17000 50  0001 C CNN
+	1    6300 17000
+	-1   0    0    1
+$EndComp
+$Comp
+L Device:R R?
+U 1 1 5C5AB4CB
+P 5800 17000
+F 0 "R?" H 5870 16954 50  0000 L CNN
+F 1 "22k" H 5870 17045 50  0000 L CNN
+F 2 "Resistor_SMD:R_0603_1608Metric_Pad1.05x0.95mm_HandSolder" V 5730 17000 50  0001 C CNN
+F 3 "~" H 5800 17000 50  0001 C CNN
+	1    5800 17000
+	-1   0    0    1
+$EndComp
+$Comp
+L power:+5V #PWR?
+U 1 1 5C692A32
+P 6300 16750
+F 0 "#PWR?" H 6300 16600 50  0001 C CNN
+F 1 "+5V" H 6315 16923 50  0000 C CNN
+F 2 "" H 6300 16750 50  0001 C CNN
+F 3 "" H 6300 16750 50  0001 C CNN
+	1    6300 16750
+	1    0    0    -1
+$EndComp
+$Comp
+L power:-5V #PWR?
+U 1 1 5C707866
+P 5800 16750
+F 0 "#PWR?" H 5800 16850 50  0001 C CNN
+F 1 "-5V" H 5815 16923 50  0000 C CNN
+F 2 "" H 5800 16750 50  0001 C CNN
+F 3 "" H 5800 16750 50  0001 C CNN
+	1    5800 16750
+	1    0    0    -1
+$EndComp
+Wire Wire Line
+	6300 16750 6300 16850
+Wire Wire Line
+	5800 16750 5800 16850
+Wire Wire Line
+	5800 17150 5800 17250
+Wire Wire Line
+	5800 17250 5900 17250
+Wire Wire Line
+	6200 17250 6300 17250
+Wire Wire Line
+	6300 17250 6300 17150
+Wire Wire Line
+	6050 17400 6050 17600
+Connection ~ 6050 17600
+Wire Notes Line
+	6600 16450 6600 17450
+Wire Notes Line
+	6600 17450 5550 17450
+Wire Notes Line
+	5550 17450 5550 16450
+Wire Notes Line
+	5550 16450 6600 16450
 $EndSCHEMATC
