File: uSensor_v1/uSensor_v1.sch (KiCad schematic (older format))
At the start: 122 parts, among them J1 +12V Supply, J2 Conn_01x03, J3 Conn_01x03, J4 NS25-W8P 6-pin 2,54mm, J5 USB_B, Q1 BC817-25T116, Q2 BC817-25T116, SW1 SW_Push, SW2 SW_Push, U1 AM10TW-2405DZ, U10 KSS-213, U11 AD7795, U12 AD5667, U13 TBD, U14 TBD, U15 REF192, U2 AZ1117-3.3, U22 RCLAMP, U3 STM32F407VGTx, U4 MCP9700AT, U5 MCP9700AT, U6 LM6132A, U7 MCP9700AT, U8 MCP9700AT, U9 UG-2864KSWLG01

Commit message: Schematic in progress.
Parts:
- removed C42, C46: 100n 6V3 X5R, Capacitor_SMD:C_0603_1608Metric_Pad1.05x0.95mm_HandSolder, symbol Device:C
- removed U13, U14: TBD, symbol Amplifier_Operational:AD8603
- added R?: 1M, Resistor_SMD:R_0603_1608Metric_Pad1.05x0.95mm_HandSolder, symbol Device:R
- added U13: TBD, symbol Amplifier_Operational:LM358
- U10: MFR (none) -> Sony; MPN (none) -> KSS-213C
- gave numbers to parts that had none: 3
Connections:
- net labels added: DAC_ADDR
- net labels removed: GNDPWR
- wire segments 639 -> 630
- no-connect marks 61 -> 62
Other:
- note added: "DC/DC CONVERTER - OK"
- note added: "EXTERNAL ADC - OK"
- note added: "EXTERNAL DAC - OK"
- note added: "OLED DISPLAY - OK"
- note added: "PCB Temperature Sensors - OK"
- note added: "SWD CONNECTOR - OK"
- note added: "TACT-SWITCH - OK"
- note added: "USB CONNECTOR - OK"
- note added: "VOLTAGE REGULATOR - OK"
- note removed: "DC/DC CONVERTER"
- note removed: "EXTERNAL ADC"
- note removed: "EXTERNAL DAC"
- note removed: "Jaka to wersja układu?\nZ referencją czy bez?"
- note removed: "Jaki zakres sygnału \nwyjściowego?"
- note removed: "OLED DISPLAY"
- note removed: "PCB Temperature Sensors"
- note removed: "SWD CONNECTOR"
- note removed: "TACT-SWITCH"
- note removed: "USB CONNECTOR"
- note removed: "VOLTAGE REGULATOR"
- moved on the sheet: C41, C45, R64, R65, RV2

Commit message: Added testpoints to schematic.
Parts:
- added TP1, TP10, TP11, TP12, TP13, TP14, TP15, TP16, TP17, TP18, TP19, TP2, TP20, TP21, TP22, TP23, TP24, TP25, TP26, TP27, TP28, TP29, TP3, TP30, TP31, TP32, TP33, TP34, TP35, TP36, TP37, TP38, TP39, TP4, TP40, TP41, TP42, TP43, TP44, TP45, TP46, TP47, TP48, TP49, TP5, TP50, TP51, TP52, TP53, TP54, TP55, TP56, TP57, TP58, TP59, TP6, TP60, TP61, TP7, TP70, TP71, TP72, TP73, TP74, TP75, TP76, TP77, TP78, TP8, TP83, TP84, TP9: TP, Sentisa-Connectors:TestPoint_Probe_1.0mmDiameter_0.6mmDrill, symbol Connector:TestPoint
- U12: footprint TBD -> Sentisa-IC:MSOP-10_4.9x3.0mm_Pitch0.5mm
- gave numbers to parts that had none: 1
Other:
- note added: "DC/DC CONVERTER"
- note added: "EXTERNAL ADC"
- note added: "EXTERNAL DAC"
- note added: "OLED DISPLAY"
- note added: "PCB Temperature Sensors"
- note added: "SWD CONNECTOR"
- note added: "TACT-SWITCH"
- note added: "TEST POINTS"
- note added: "USB CONNECTOR"
- note added: "VOLTAGE REGULATOR"
- note removed: "DC/DC CONVERTER - OK"
- note removed: "EXTERNAL ADC - OK"
- note removed: "EXTERNAL DAC - OK"
- note removed: "OLED DISPLAY - OK"
- note removed: "PCB Temperature Sensors - OK"
- note removed: "SWD CONNECTOR - OK"
- note removed: "TACT-SWITCH - OK"
- note removed: "USB CONNECTOR - OK"
- note removed: "VOLTAGE REGULATOR - OK"
- moved on the sheet: C25, C26, C27, C28, C29, C30, C35, C36, R18, R19, U10, U9

Commit message: Added OLED FP.
Parts:
- U9: footprint TBD -> Sentisa-IC:UG-2864KSWLG01
Changed lines of the file:
@@
 F 0 "U9" H 19050 7650 50  0000 C CNN
 F 1 "UG-2864KSWLG01" H 18450 7650 50  0000 C CNN
-F 2 "TBD" H 18700 6050 50  0001 C CNN
+F 2 "Sentisa-IC:UG-2864KSWLG01" H 18700 6050 50  0001 C CNN
 F 3 "" H 18700 6050 50  0001 C CNN
 F 4 "WiseChip" H 18600 6050 50  0001 C CNN "MFR"

Commit message: Schematic in progress.
Parts:
- removed TP20: TP, Sentisa-Connectors:TestPoint_Probe_1.0mmDiameter_0.6mmDrill, symbol Connector:TestPoint
- Q1, Q2: value BC817-25T116 -> BC817-25; footprint TBD -> Sentisa-IC:SOT-23_o1; symbol Device:Q_NPN_BCE -> Device:Q_NPN_BEC; MFR (none) -> Diotec Semiconductor; MPN (none) -> BC817-25
- U3: footprint Package_QFP:LQFP-100_14x14mm_P0.5mm -> Sentisa-Microcontrollers:ST_S-LQFP-100_14x14mm_P0.5mm
Connections:
- net +3V3: now also TP1.1
- net +5V: now also Q1.3 (C), Q2.3 (C), TP2.1; no longer Q1.2 (C), Q2.2 (C)
- net -5V: now also TP5.1
- net ADC_DIN: now also TP48.1
- net ADC_DOUT: now also TP49.1
- net ADC_SCLK: now also TP47.1
- net ADC_~CS: now also TP46.1
- net COIL_F+: now also TP38.1
- net COIL_F-: now also TP37.1
- net COIL_T+: now also TP35.1
- net COIL_T-: now also TP36.1
- net DAC_ADDR: now also TP28.1
- net DAC_LD_CTRL: now also TP72.1
- net DAC_OUT_COIL_F_CTRL: now also TP32.1
- net DAC_OUT_COIL_T_CTRL: now also TP31.1
- net DAC_SCL: now also TP30.1
- net DAC_SDA: now also TP29.1
- net DAC_~CLR: now also TP27.1
- net FOC_ERR_2_ADC: now also TP58.1
- net LCD_A0: now also TP10.1
- net LCD_CS: now also TP6.1
- net LCD_RST: now also TP7.1
- net LCD_SCK: now also TP11.1
- net LCD_SI: now also TP14.1
- net REF_2.5V: now also TP59.1
- net SENS_A: now also TP41.1
- net SENS_B: now also TP42.1
- net SENS_C: now also TP43.1
- net SENS_D: now also TP44.1
- net SENS_IN_AMP_A/SENS_OUT: now also TP52.1
- net SENS_IN_AMP_B/SENS_OUT: now also TP56.1
- net SENS_IN_AMP_C/SENS_OUT: now also TP60.1
- net SENS_IN_AMP_D/SENS_OUT: now also TP57.1, TP61.1
- net SENS_LD: now also TP40.1
- net SENS_LD_PWR: now also TP71.1
- net SENS_PD: now also TP39.1
- net SENS_PD_ADC: now also TP70.1
- net SWITCH_1: now also TP17.1
- net SWITCH_2: now also TP15.1
- net TEMP_SENS_OUT_1: now also TP23.1
- net TEMP_SENS_OUT_2: now also TP25.1
- net TEMP_SENS_OUT_3: now also TP24.1
- net TEMP_SENS_OUT_4: now also TP26.1
- net at R3.1, R4.1, U6.1: now also TP75.1
- net at R1.1, R2.1, R3.2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: now also TP77.1
- net at J3.3 (Pin_3), R5.1, U6.3 (+): now also TP73.1
- net at C1.2, R4.2, U6.6 (-): now also TP78.1
- net at C1.1, Q2.1 (B), U6.7: now also TP76.1
- net at R12.1: now also Q2.2 (E); no longer Q2.3 (E)
- net at C25.2, U9.2 (C2P): now also TP8.1
- net at R18.1, U9.26 (IREF): now also TP16.1
- net at C36.1, U9.27 (VCOMH): now also TP18.1
- net at C35.1, U9.28 (VCC): now also TP19.1
- net at C25.1, U9.3 (C2N): now also TP9.1
- net at C26.2, U9.4 (C1P): now also TP12.1
- net at C26.1, U9.5 (C1N): now also TP13.1
- net at TP3.1: now also D1.2 (A), J1.1 (Pin_1)
- net at C11.2, C12.2, D3.2 (A2)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: now also TP4.1
- net at TP21.1: now also R9.1, U3.97 (PE0/TIM4_ETR/FSMC_NBL0/DCMI_D2/EVENTOUT)
- net at TP22.1: now also R10.1, U3.98 (PE1/FSMC_NBL1/DCMI_D3/EVENTOUT)
- net at R26.1, R30.1, R32.1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: now also TP50.1
- net at R27.1, R28.1, R33.2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: now also TP53.1
- net at TP34.1: now also U10.3 (E)
- net at TP45.1: now also U10.8 (F)
- net at TP33.1: now also R19.1, U10.11 (VR)
- net at R31.1, U13.6 (-), U13.7: now also TP55.1
- net at R26.2, R29.1, U13.1: now also TP51.1
- net at C43.2, R29.2, U13.5 (+): now also TP54.1
- net at RV1.2, U6.5 (+): now also TP74.1
- net at TP83.1: now also Q1.1 (B), R11.2, R8.1
- net at R13.1: now also Q1.2 (E); no longer Q1.3 (E)
- no-connect marks 62 -> 60
Other:
- moved on the sheet: C18, C20, C67, RV1, TP15, TP17, TP23, TP24, TP25, TP26, TP34, TP35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

Commit message: Schematic checked.
Parts:
- added C?: 10u, Capacitor_SMD:C_0603_1608Metric_Pad1.05x0.95mm_HandSolder, symbol Device:C
- added L?: 1u w 1210, symbol Device:L
- L1, L3: value 100u 1A -> 10u 1A; MFR Ferrocore -> TBD; MPN DLG-1005-101 -> TBD
- R12, R13: value 33R -> 0R; footprint TBD -> Sentisa-Resistors:R_1206
- R19: footprint TBD -> Sentisa-Resistors:R_0603
- U2: value AZ1117-3.3 -> TBD
Connections:
- net GND: now also C?.2
- net SENS_LD: now also L?.1; no longer U10.10 (LD)
- new net: C?.1, L?.2, U10.10 (LD)
Other:
- note added: "Dać rezonator"
- note added: "Zmiana"
Changed lines of the file:
@@
 Text GLabel 4750 14600 2    50   Input ~ 0
 SENS_B
-Text GLabel 2500 14500 0    50   Input ~ 0
+Text GLabel 1050 13800 0    50   Input ~ 0
 SENS_LD
 Text GLabel 2100 14900 0    50   Input ~ 0
@@
 F 0 "R19" H 1070 14996 50  0000 L CNN
 F 1 "TBD" H 1070 14905 50  0000 L CNN
-F 2 "TBD" V 930 14950 50  0001 C CNN
+F 2 "Sentisa-Resistors:R_0603" V 930 14950 50  0001 C CNN
 F 3 "~" H 1000 14950 50  0001 C CNN
 	1    1000 14950
@@
 P 6000 2950
 F 0 "L3" V 5914 2950 50  0000 C CNN
-F 1 "100u 1A" V 5823 2950 50  0000 C CNN
+F 1 "10u 1A" V 5823 2950 50  0000 C CNN
 F 2 "Sentisa-Coils:FERROCORE_DLG-1005-101" H 6000 2950 50  0001 C CNN
 F 3 "~" H 6000 2950 50  0001 C CNN
-F 4 "Ferrocore" V 6000 2950 50  0001 C CNN "MFR"
-F 5 "DLG-1005-101" V 6000 2950 50  0001 C CNN "MPN"
+F 4 "TBD" V 6000 2950 50  0001 C CNN "MFR"
+F 5 "TBD" V 6000 2950 50  0001 C CNN "MPN"
 	1    6000 2950
 	0    -1   -1   0
@@
 P 6000 1750
 F 0 "L1" V 6190 1750 50  0000 C CNN
-F 1 "100u 1A" V 6099 1750 50  0000 C CNN
+F 1 "10u 1A" V 6099 1750 50  0000 C CNN
 F 2 "Sentisa-Coils:FERROCORE_DLG-1005-101" H 6000 1750 50  0001 C CNN
 F 3 "~" H 6000 1750 50  0001 C CNN
-F 4 "Ferrocore" V 6000 1750 50  0001 C CNN "MFR"
-F 5 "DLG-1005-101" V 6000 1750 50  0001 C CNN "MPN"
+F 4 "TBD" V 6000 1750 50  0001 C CNN "MFR"
+F 5 "TBD" V 6000 1750 50  0001 C CNN "MPN"
 	1    6000 1750
 	0    -1   -1   0
@@
 	2700 15100 2800 15100
 Wire Wire Line
-	2500 14500 2800 14500
-Wire Wire Line
 	4750 14600 4200 14600
 Wire Wire Line
@@
 P 9150 1300
 F 0 "U2" H 9150 1542 50  0000 C CNN
-F 1 "AZ1117-3.3" H 9150 1451 50  0000 C CNN
+F 1 "TBD" H 9150 1451 50  0000 C CNN
 F 2 "Package_TO_SOT_SMD:SOT-223-3_TabPin2" H 9150 1550 50  0001 C CIN
 F 3 "https://www.diodes.com/assets/Datasheets/AZ1117.pdf" H 9150 1300 50  0001 C CNN
@@
 P 5050 26200
 F 0 "R12" H 4980 26246 50  0000 R CNN
-F 1 "33R" H 4980 26155 50  0000 R CNN
-F 2 "TBD" V 4980 26200 50  0001 C CNN
+F 1 "0R" H 4980 26155 50  0000 R CNN
+F 2 "Sentisa-Resistors:R_1206" V 4980 26200 50  0001 C CNN
 F 3 "~" H 5050 26200 50  0001 C CNN
 	1    5050 26200
@@
 P 7550 26200
 F 0 "R13" H 7480 26246 50  0000 R CNN
-F 1 "33R" H 7480 26155 50  0000 R CNN
-F 2 "TBD" V 7480 26200 50  0001 C CNN
+F 1 "0R" H 7480 26155 50  0000 R CNN
+F 2 "Sentisa-Resistors:R_1206" V 7480 26200 50  0001 C CNN
 F 3 "~" H 7550 26200 50  0001 C CNN
 	1    7550 26200
@@
 Wire Wire Line
 	10500 8850 10400 8850
-$Comp
-L power:+5V #PWR0107
-U 1 1 69068D29
-P 6100 13500
-F 0 "#PWR0107" H 6100 13350 50  0001 C CNN
-F 1 "+5V" H 6115 13673 50  0000 C CNN
-F 2 "" H 6100 13500 50  0001 C CNN
-F 3 "" H 6100 13500 50  0001 C CNN
-	1    6100 13500
-	1    0    0    -1
-$EndComp
 Text GLabel 6450 14650 0    50   Input ~ 0
 REF_2.5V
@@
 	12800 3950 12800 3850
 Wire Wire Line
-	12800 3850 13300 3850
-Wire Wire Line
 	10400 7350 10500 7350
 Wire Wire Line
@@
 FT
 NoConn ~ 13600 5450
-Wire Wire Line
-	13600 5350 13300 5350
-Wire Wire Line
-	13300 5350 13300 3850
-Connection ~ 13300 3850
-Wire Wire Line
-	13300 3850 13900 3850
 Text GLabel 12600 15100 0    50   Input ~ 0
 FOC_ERR_2_ADC
@@
 Wire Wire Line
 	7900 17000 7800 17000
-Wire Notes Line
-	8850 16450 7300 16450
-Wire Notes Line
-	7300 17500 8850 17500
-Wire Notes Line
-	8850 17500 8850 16450
 Text Notes 10400 8750 0    50   ~ 0
 FT
@@
 Wire Wire Line
 	7300 20200 7300 20100
-Wire Notes Line
-	7300 16450 7300 17500
 $Comp
 L Device:R R66
@@
 	0    -1   1    0
 $EndComp
-Text Notes 7750 16850 2    250  ~ 50
-?
 Wire Wire Line
 	7500 17000 6050 17000
@@
 Text Notes 7850 25600 0    150  ~ 30
 ?
+Wire Wire Line
+	12800 3850 13300 3850
+Wire Wire Line
+	13600 5350 13300 5350
+Wire Wire Line
+	13300 5350 13300 3850
+Connection ~ 13300 3850
+Wire Wire Line
+	13300 3850 13900 3850
+$Comp
+L Device:L L?
+U 1 1 5C93A5EF
+P 1500 13800
+F 0 "L?" V 1690 13800 50  0000 C CNN
+F 1 "1u w 1210" V 1599 13800 50  0000 C CNN
+F 2 "" H 1500 13800 50  0001 C CNN
+F 3 "~" H 1500 13800 50  0001 C CNN
+	1    1500 13800
+	0    -1   -1   0
+$EndComp
+$Comp
+L Device:C C?
+U 1 1 5C93A9EE
+P 1750 14050
+F 0 "C?" H 1635 14096 50  0000 R CNN
+F 1 "10u" H 1635 14005 50  0000 R CNN
+F 2 "Capacitor_SMD:C_0603_1608Metric_Pad1.05x0.95mm_HandSolder" H 1788 13900 50  0001 C CNN
+F 3 "~" H 1750 14050 50  0001 C CNN
+	1    1750 14050
+	1    0    0    -1
+$EndComp
+Wire Wire Line
+	1750 13900 1750 13800
+Wire Wire Line
+	1750 13800 1650 13800
+Wire Wire Line
+	1350 13800 1050 13800
+$Comp
+L power:GND #PWR?
+U 1 1 5CA5CFBF
+P 1750 14300
+F 0 "#PWR?" H 1750 14050 50  0001 C CNN
+F 1 "GND" H 1755 14127 50  0000 C CNN
+F 2 "" H 1750 14300 50  0001 C CNN
+F 3 "" H 1750 14300 50  0001 C CNN
+	1    1750 14300
+	1    0    0    -1
+$EndComp
+Wire Wire Line
+	1750 14200 1750 14300
+Wire Wire Line
+	2800 14500 2250 14500
+Wire Wire Line
+	2250 14500 2250 13800
+Wire Wire Line
+	2250 13800 1750 13800
+Connection ~ 1750 13800
+Wire Notes Line
+	10800 16800 12350 16800
+Wire Notes Line
+	12350 16800 12350 17900
+Wire Notes Line
+	12350 17900 10800 17900
+Wire Notes Line
+	10800 17900 10800 16800
+Text Notes 11250 17300 0    50   ~ 0
+Dać rezonator
+Text Notes 10150 1400 0    150  ~ 30
+Zmiana
 $EndSCHEMATC

Commit message: Schematic in progress.
Parts:
- added C46, C68, C69, C70: 100n 6V3 X5R, Capacitor_SMD:C_0603_1608Metric_Pad1.05x0.95mm_HandSolder, symbol Device:C
- added J6: GNDA-GNDD Jumper, Connector_PinHeader_2.54mm:PinHeader_1x02_P2.54mm_Vertical, symbol Connector_Generic:Conn_01x02
- added R67, R68, R69, R70: 10k, Resistor_SMD:R_0603_1608Metric_Pad1.05x0.95mm_HandSolder, symbol Device:R
- added R71, R72: 10k N.M., Resistor_SMD:R_0603_1608Metric_Pad1.05x0.95mm_HandSolder, symbol Device:R
- added TP20, TP85, TP86, TP87, TP88, TP89, TP90, TP91, TP92, TP93, TP94, TP95, TP96, TP97, TP98, TP99: TP, Sentisa-Connectors:TestPoint_Probe_1.0mmDiameter_0.6mmDrill, symbol Connector:TestPoint
- C2: value 10u 6V3 X5R -> 100n 6V3 X5R
- C3: value 22u 6V3 X5R -> 10u 6V3 X5R
- C42: renamed from C?; value 10u -> 10u 10V X5R
- L1, L3: value 10u 1A -> 82u 1A; footprint Sentisa-Coils:FERROCORE_DLG-1005-101 -> Inductor_SMD:L_1210_3225Metric_Pad1.42x2.65mm_HandSolder; MFR TBD -> Fastron; MPN TBD -> 1210AS-082J-01
- L4: renamed from L?; value 1u w 1210 -> 10u; footprint (none) -> Inductor_SMD:L_1210_3225Metric_Pad1.42x2.65mm_HandSolder; MFR (none) -> TDK; MPN (none) -> NLCV32T-100K-EF
- R1: value 220k -> 220k 1%
- R2: value 220R -> 220R 1%
- R26, R29, R33: value 150k -> 150k 1%
- R27, R28, R3, R30, R32: value 10k -> 10k 1%
- R31: value 51R -> 51R 1%
- R4: value 22k -> 22k 1%
- R5: value 100R -> 100R 1%
- U10: footprint TBD -> TBD -> Marcel
- U13: footprint (none) -> Sentisa-IC:SO-8; MFR TBD -> Diodes Incorporated; MPN TBD -> AZ4580MTR-G1
- U2: value TBD -> LD1117A; footprint Package_TO_SOT_SMD:SOT-223-3_TabPin2 -> Sentisa-IC:TO-252-2; MFR Diodes Incorporated -> ST; MPN AZ1117CH-3.3TRG1 -> LD1117ADT33TR
- U9: footprint Sentisa-IC:UG-2864KSWLG01 -> Sentisa-IC:UG-2864KSWLG01_Adhessive_Tape_Flat_Mounting
Connections:
- net ADC_~CS: now also R72.2
- net GNDA: now also C10.2, C14.1, C15.1, C19.2, C29.2, C30.2, C31.2, C32.2, C41.2, C42.2, C43.1, C44.2, C45.2, C47.2, C48.2, C49.2, C50.2, C9.2, D2.2 (A2), D4.1 (A1), R11.1, R19.2, R2.2, R33.1, R5.2, R6.2, RV1.3, TP84.1, U1.16 (Common), U1.9 (Common), U10.9 (GND), U11.10 (AIN2(-)), U11.12 (AIN3(-)), U11.14 (REFIN1(-)), U11.16 (AIN5(-)/IOUT1), U11.18 (AIN4(-)/REFIN2(-)), U11.20 (GND), U11.6 (AIN6(-)/P2), U11.8 (AIN1(-)), U15.4 (GND), U6.4 (V-), C46.2, C68.2, C69.2, C70.2, J6.1 (Pin_1), TP20.1, TP85.1, TP86.1, TP87.1, TP88.1, TP89.1, TP90.1
- net GNDD: now also C13.2, C16.2, C17.2, C18.2, C2.2, C20.2, C21.2, C22.2, C23.2, C24.2, C27.1, C28.1, C3.2, C33.2, C34.2, C35.2, C36.2, C37.2, C38.2, C39.2, C4.2, C40.2, C5.2, C6.2, C67.2, C7.2, C8.2, D5.1 (K), D6.1 (K), J4.3 (Pin_3), J5.4 (GND), J5.5 (Shield), R18.2, R7.2, SW1.2, SW2.2, U12.3 (GND), U2.1 (GND), U22.2 (GND), U3.10 (VSS), U3.20 (VSSA), U3.27 (VSS), U3.74 (VSS), U3.99 (VSS), U4.3 (GND), U5.3 (GND), U7.3 (GND), U8.3 (GND), U9.10 (BS0), U9.11 (BS1), U9.12 (BS2), U9.16 (R/W#), U9.17 (E/RD#), U9.20 (D2), U9.21 (D3), U9.22 (D4), U9.23 (D5), U9.24 (D6), U9.25 (D7), U9.29 (VLSS), U9.8 (VSS), J6.2 (Pin_2), R71.1, R72.1, TP91.1, TP92.1, TP93.1, TP94.1, TP95.1, TP96.1, TP97.1, TP98.1
- net SENS_A: now also R67.1; no longer U11.9 (AIN2(+))
- net SENS_B: now also R68.1; no longer U11.11 (AIN3(+))
- net SENS_C: now also R69.1; no longer U11.17 (AIN4(+)/REFIN2(+))
- net SENS_D: now also R70.1; no longer U11.15 (AIN5(+)/IOUT2)
- net at U11.2 (CLK): now also TP99.1
- net DAC_~LDAC: now reaches U3.91 (I2C1_SMBA/CAN2_RX/OTG_HS_ULPI_D7/ETH_PPS_OUT/TIM3_CH2/SPI1_MOSI/SPI3_MOSI/DCMI_D10/I2S3_SD/EVENTOUT/PB5)
- net DAC_~LDAC: now also U12.4 (~LDAC), R71.2
- removed net GND: C10.2, C13.2, C14.1, C15.1, C16.2, C17.2, C18.2, C19.2, C2.2, C20.2, C21.2, C22.2, C23.2, C24.2, C27.1, C28.1, C29.2, C3.2, C30.2, C31.2, C32.2, C33.2, C34.2, C35.2, C36.2, C37.2, C38.2, C39.2, C4.2, C40.2, C41.2, C42.2, C43.1, C44.2, C45.2, C47.2, C48.2, C49.2, C5.2, C50.2, C6.2, C67.2, C7.2, C8.2, C9.2, D2.2 (A2), D4.1 (A1), D5.1 (K), D6.1 (K), J4.3 (Pin_3), J5.4 (GND), J5.5 (Shield), R11.1, R18.2, R19.2, R2.2, R33.1, R5.2, R6.2, R7.2, RV1.3, SW1.2, SW2.2, U1.16 (Common), U1.9 (Common), U10.9 (GND), U11.10 (AIN2(-)), U11.12 (AIN3(-)), U11.14 (REFIN1(-)), U11.16 (AIN5(-)/IOUT1), U11.18 (AIN4(-)/REFIN2(-)), U11.20 (GND), U11.6 (AIN6(-)/P2), U11.8 (AIN1(-)), U12.3 (GND), U12.4 (~LDAC), U15.4 (GND), U2.1 (GND), U22.2 (GND), U3.10 (VSS), U3.20 (VSSA), U3.27 (VSS), U3.74 (VSS), U3.99 (VSS), U4.3 (GND), U5.3 (GND), U6.4 (V-), U7.3 (GND), U8.3 (GND), U9.10 (BS0), U9.11 (BS1), U9.12 (BS2), U9.16 (R/W#), U9.17 (E/RD#), U9.20 (D2), U9.21 (D3), U9.22 (D4), U9.23 (D5), U9.24 (D6), U9.25 (D7), U9.29 (VLSS), U9.8 (VSS)
- new net: C46.1, R67.2, U11.9 (AIN2(+))
- new net: C68.1, R68.2, U11.11 (AIN3(+))
- new net: C69.1, R69.2, U11.17 (AIN4(+)/REFIN2(+))
- new net: C70.1, R70.2, U11.15 (AIN5(+)/IOUT2)
- no-connect marks 60 -> 58
Other:
- note added: "COIL CURRENT SOURCES - NOK"
- note added: "DC/DC CONVERTER - OK"
- note added: "Dodać rezonator"
- note added: "EXTERNAL ADC - NOK"
- note added: "EXTERNAL DAC - OK"
- note added: "LASER CURRENT SOURCE - OK"
- note added: "MCU - OK"
- note added: "OLED DISPLAY - OK"
- note added: "PCB Temperature Sensors - OK"
- note added: "PICKUP KSS-213 - NOK"
- note added: "PWR FLAGS - OK"
- note added: "SENSORS SINGALS SUMMING CIRCUIT - NOK"
- note added: "SWD CONNECTOR - OK"
- note added: "TACT-SWITCH - OK"
- note added: "USB CONNECTOR - OK"
- note added: "VOLTAGE REGULATOR - OK"
- note removed: "?"
- note removed: "COIL CURRENT SOURCES"
- note removed: "DC/DC CONVERTER"
- note removed: "Dać rezonator"
- note removed: "EXTERNAL ADC"
- note removed: "EXTERNAL DAC"
- note removed: "LASER CURRENT SOURCE"
- note removed: "MCU"
- note removed: "OLED DISPLAY"
- note removed: "PCB Temperature Sensors"
- note removed: "PICKUP KSS-213"
- note removed: "PWR FLAGS"
- note removed: "SENSORS SINGALS SUMMING CIRCUIT"
- note removed: "SWD CONNECTOR"
- note removed: "TACT-SWITCH"
- note removed: "USB CONNECTOR"
- note removed: "VOLTAGE REGULATOR"
- note removed: "Zmiana"
- moved on the sheet: C25, C26, C27, C28, C29, C30, C31, C32, C33, C34, C35, C36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
