File: uSensor_v1/uSensor_v1.sch (KiCad schematic (older format))
At the start: 220 parts, among them J1 +12V Supply, J2 Conn_01x03, J3 Conn_01x03, J4 NS25-W8P 6-pin 2,54mm, J5 USB_B, J6 GNDA-GNDD Jumper, Q1 BC817-25, Q2 BC817-25, SW1 SW_Push, SW2 SW_Push, U1 AM10TW-2405DZ, U10 KSS-213, U11 AD7795, U12 AD5667, U13 TBD, U15 REF192, U2 LD1117A, U22 RCLAMP, U3 STM32F407VGTx, U4 MCP9700AT, U5 MCP9700AT, U6 LM6132A, U7 MCP9700AT, U8 MCP9700AT, U9 UG-2864KSWLG01

Commit message: Layout in progress.
Parts:
- added C71, C72: 100n 6V3 X5R, Capacitor_SMD:C_0603_1608Metric_Pad1.05x0.95mm_HandSolder, symbol Device:C
- added R73, R74: 10k, Resistor_SMD:R_0603_1608Metric_Pad1.05x0.95mm_HandSolder, symbol Device:R
- C1: value 1n -> 1n 16V X5R
- D2, D4: footprint Sentisa-Diodes:D_SOD-523 -> Sentisa-Diodes:D_SMB; MFR On Semiconductor -> Vishay; MPN ESD5Z7.0T1G -> SMBJ7.0D-M3/H
- U13: footprint Sentisa-IC:SO-8 -> TBD; MFR Diodes Incorporated -> TBD; MPN AZ4580MTR-G1 -> TBD
Connections:
- net FOC_ERR_2_ADC: now also R73.1; no longer U11.7 (AIN1(+))
- net GNDA: now also C71.2, C72.2
- net SENS_PD: now also R74.1; no longer U11.5 (AIN6(+)/P1)
- net USB_D+: now also U22.1 (D1); no longer U22.3 (D2)
- net USB_D-: now also U22.3 (D2); no longer U22.1 (D1)
- new net: C71.1, R73.2, U11.7 (AIN1(+))
- new net: C72.1, R74.2, U11.5 (AIN6(+)/P1)
Changed lines of the file:
@@
 P 4150 26550
 F 0 "C1" V 4310 26550 50  0000 C CNN
-F 1 "1n" V 4401 26550 50  0000 C CNN
+F 1 "1n 16V X5R" V 4401 26550 50  0000 C CNN
 F 2 "Capacitor_SMD:C_0603_1608Metric_Pad1.05x0.95mm_HandSolder" H 4188 26400 50  0001 C CNN
 F 3 "~" H 4150 26550 50  0001 C CNN
@@
 F 0 "D4" V 6954 2729 50  0000 L CNN
 F 1 "TVS 7V" V 7045 2729 50  0000 L CNN
-F 2 "Sentisa-Diodes:D_SOD-523" H 7000 2450 50  0001 C CNN
+F 2 "Sentisa-Diodes:D_SMB" H 7000 2450 50  0001 C CNN
 F 3 "" H 6950 2650 50  0001 C CNN
-F 4 "On Semiconductor" V 7000 2650 50  0001 C CNN "MFR"
-F 5 "ESD5Z7.0T1G" V 7000 2650 50  0001 C CNN "MPN"
+F 4 "Vishay" V 7000 2650 50  0001 C CNN "MFR"
+F 5 "SMBJ7.0D-M3/H" V 7000 2650 50  0001 C CNN "MPN"
 	1    7000 2650
 	0    1    1    0
@@
 F 0 "D2" V 6954 2129 50  0000 L CNN
 F 1 "TVS 7V" V 7045 2129 50  0000 L CNN
-F 2 "Sentisa-Diodes:D_SOD-523" H 7000 1850 50  0001 C CNN
+F 2 "Sentisa-Diodes:D_SMB" H 7000 1850 50  0001 C CNN
 F 3 "" H 6950 2050 50  0001 C CNN
-F 4 "On Semiconductor" V 7000 2050 50  0001 C CNN "MFR"
-F 5 "ESD5Z7.0T1G" V 7000 2050 50  0001 C CNN "MPN"
+F 4 "Vishay" V 7000 2050 50  0001 C CNN "MFR"
+F 5 "SMBJ7.0D-M3/H" V 7000 2050 50  0001 C CNN "MPN"
 	1    7000 2050
 	0    1    1    0
@@
 USB_VBUS
 Wire Wire Line
-	13200 4450 13500 4450
-Wire Wire Line
-	13200 4150 13400 4150
-Wire Wire Line
 	12600 4250 12800 4250
 Wire Wire Line
@@
 	13600 5150 13500 5150
 Wire Wire Line
-	13500 5150 13500 4450
-Connection ~ 13500 4450
-Wire Wire Line
-	13500 4450 13900 4450
-Wire Wire Line
 	13600 5250 13400 5250
-Wire Wire Line
-	13400 5250 13400 4150
-Connection ~ 13400 4150
-Wire Wire Line
-	13400 4150 13900 4150
 Wire Notes Line
 	11950 3200 14950 3200
@@
 FT
 NoConn ~ 13600 5450
-Text GLabel 14650 14950 0    50   Input ~ 0
+Text GLabel 12750 13850 0    50   Input ~ 0
 FOC_ERR_2_ADC
 $Comp
@@
 	14750 16250 14750 15950
 Connection ~ 14750 15950
-Text GLabel 14500 16450 0    50   Input ~ 0
+Text GLabel 12450 16450 0    50   Input ~ 0
 SENS_PD
 Wire Wire Line
-	14500 16450 14850 16450
-Wire Wire Line
 	14750 16250 14750 16550
 Wire Wire Line
@@
 Wire Wire Line
 	14750 14750 14850 14750
-Wire Wire Line
-	14850 14950 14650 14950
 Text Notes 10400 8850 0    50   ~ 0
 FT
@@
 F 0 "U13" H 6750 18350 50  0000 C CNN
 F 1 "TBD" H 6800 18050 50  0000 C CNN
-F 2 "Sentisa-IC:SO-8" H 6550 18200 50  0001 C CNN
-F 3 "https://pl.mouser.com/datasheet/2/115/AZ4580-271600.pdf" H 6550 18200 50  0001 C CNN
-F 4 "Diodes Incorporated" H 6550 18200 50  0001 C CNN "MFR"
-F 5 "AZ4580MTR-G1" H 6550 18200 50  0001 C CNN "MPN"
+F 2 "TBD" H 6550 18200 50  0001 C CNN
+F 3 "" H 6550 18200 50  0001 C CNN
+F 4 "TBD" H 6550 18200 50  0001 C CNN "MFR"
+F 5 "TBD" H 6550 18200 50  0001 C CNN "MPN"
 	1    6550 18200
 	1    0    0    -1
@@
 F 0 "U13" H 8300 18667 50  0000 C CNN
 F 1 "TBD" H 8300 18576 50  0000 C CNN
-F 2 "Sentisa-IC:SO-8" H 8300 18300 50  0001 C CNN
-F 3 "https://pl.mouser.com/datasheet/2/115/AZ4580-271600.pdf" H 8300 18300 50  0001 C CNN
-F 4 "Diodes Incorporated" H 8300 18300 50  0001 C CNN "MFR"
-F 5 "AZ4580MTR-G1" H 8300 18300 50  0001 C CNN "MPN"
+F 2 "TBD" H 8300 18300 50  0001 C CNN
+F 3 "" H 8300 18300 50  0001 C CNN
+F 4 "TBD" H 8300 18300 50  0001 C CNN "MFR"
+F 5 "TBD" H 8300 18300 50  0001 C CNN "MPN"
 	2    8300 18300
 	1    0    0    -1
@@
 F 0 "U13" H 7358 19846 50  0000 L CNN
 F 1 "TBD" H 7358 19755 50  0000 L CNN
-F 2 "Sentisa-IC:SO-8" H 7400 19800 50  0001 C CNN
-F 3 "https://pl.mouser.com/datasheet/2/115/AZ4580-271600.pdf" H 7400 19800 50  0001 C CNN
-F 4 "Diodes Incorporated" H 7400 19800 50  0001 C CNN "MFR"
-F 5 "AZ4580MTR-G1" H 7400 19800 50  0001 C CNN "MPN"
+F 2 "TBD" H 7400 19800 50  0001 C CNN
+F 3 "" H 7400 19800 50  0001 C CNN
+F 4 "TBD" H 7400 19800 50  0001 C CNN "MFR"
+F 5 "TBD" H 7400 19800 50  0001 C CNN "MPN"
 	3    7400 19800
 	1    0    0    -1
@@
 Connection ~ 1750 13850
 Wire Notes Line
-	12450 16650 14000 16650
+	12450 17600 14000 17600
 Wire Notes Line
-	14000 16650 14000 17750
+	14000 17600 14000 18700
 Wire Notes Line
-	14000 17750 12450 17750
+	14000 18700 12450 18700
 Wire Notes Line
-	12450 17750 12450 16650
+	12450 18700 12450 17600
 $Comp
 L Device:C C46
@@
 Wire Wire Line
 	14750 16750 14850 16750
-Text Notes 12850 17250 0    50   ~ 0
+Text Notes 12850 18200 0    50   ~ 0
 Dodać rezonator
+$Comp
+L Device:C C71
+U 1 1 5FD0B84B
+P 13250 14100
+F 0 "C71" H 13135 14146 50  0000 R CNN
+F 1 "100n 6V3 X5R" H 13135 14055 50  0000 R CNN
+F 2 "Capacitor_SMD:C_0603_1608Metric_Pad1.05x0.95mm_HandSolder" H 13288 13950 50  0001 C CNN
+F 3 "~" H 13250 14100 50  0001 C CNN
+	1    13250 14100
+	1    0    0    -1
+$EndComp
+$Comp
+L Device:R R73
+U 1 1 5FD0B852
+P 13000 13850
+F 0 "R73" V 13207 13850 50  0000 C CNN
+F 1 "10k" V 13116 13850 50  0000 C CNN
+F 2 "Resistor_SMD:R_0603_1608Metric_Pad1.05x0.95mm_HandSolder" V 12930 13850 50  0001 C CNN
+F 3 "~" H 13000 13850 50  0001 C CNN
+	1    13000 13850
+	0    -1   -1   0
+$EndComp
+Wire Wire Line
+	13150 13850 13250 13850
+Wire Wire Line
+	13250 13850 13250 13950
+$Comp
+L power:GNDA #PWR076
+U 1 1 5FD0B85B
+P 13250 14350
+F 0 "#PWR076" H 13250 14100 50  0001 C CNN
+F 1 "GNDA" H 13255 14177 50  0000 C CNN
+F 2 "" H 13250 14350 50  0001 C CNN
+F 3 "" H 13250 14350 50  0001 C CNN
+	1    13250 14350
+	1    0    0    -1
+$EndComp
+Wire Wire Line
+	13250 14350 13250 14250
+Wire Wire Line
+	12850 13850 12750 13850
+Wire Wire Line
+	13450 14950 13450 13850
+Wire Wire Line
+	13450 13850 13250 13850
+Wire Wire Line
+	13450 14950 14850 14950
+Connection ~ 13250 13850
+$Comp
+L Device:C C72
+U 1 1 60182D75
+P 12950 16700
+F 0 "C72" H 12835 16746 50  0000 R CNN
+F 1 "100n 6V3 X5R" H 12835 16655 50  0000 R CNN
+F 2 "Capacitor_SMD:C_0603_1608Metric_Pad1.05x0.95mm_HandSolder" H 12988 16550 50  0001 C CNN
+F 3 "~" H 12950 16700 50  0001 C CNN
+	1    12950 16700
+	1    0    0    -1
+$EndComp
+$Comp
+L Device:R R74
+U 1 1 60182D7C
+P 12700 16450
+F 0 "R74" V 12907 16450 50  0000 C CNN
+F 1 "10k" V 12816 16450 50  0000 C CNN
+F 2 "Resistor_SMD:R_0603_1608Metric_Pad1.05x0.95mm_HandSolder" V 12630 16450 50  0001 C CNN
+F 3 "~" H 12700 16450 50  0001 C CNN
+	1    12700 16450
+	0    -1   -1   0
+$EndComp
+Wire Wire Line
+	12850 16450 12950 16450
+Wire Wire Line
+	12950 16450 12950 16550
+$Comp
+L power:GNDA #PWR077
+U 1 1 60182D85
+P 12950 16950
+F 0 "#PWR077" H 12950 16700 50  0001 C CNN
+F 1 "GNDA" H 12955 16777 50  0000 C CNN
+F 2 "" H 12950 16950 50  0001 C CNN
+F 3 "" H 12950 16950 50  0001 C CNN
+	1    12950 16950
+	1    0    0    -1
+$EndComp
+Wire Wire Line
+	12950 16950 12950 16850
+Wire Wire Line
+	12550 16450 12450 16450
+Connection ~ 12950 16450
+Wire Wire Line
+	12950 16450 14850 16450
+Wire Wire Line
+	13200 4450 13400 4450
+Wire Wire Line
+	13200 4150 13500 4150
+Wire Wire Line
+	13500 5150 13500 4150
+Connection ~ 13500 4150
+Wire Wire Line
+	13500 4150 13900 4150
+Wire Wire Line
+	13400 5250 13400 4450
+Connection ~ 13400 4450
+Wire Wire Line
+	13400 4450 13900 4450
 $EndSCHEMATC

Commit message: Before schematic changing.
Parts:
- U13: footprint TBD -> Sentisa-IC:SO-8
Changed lines of the file:
@@
 Text GLabel 8400 14650 2    50   Output ~ 0
 DAC_OUT_COIL_F_CTRL
-Text GLabel 3350 30000 2    50   Input ~ 0
+Text GLabel 3400 29800 2    50   Input ~ 0
 COIL_T+
-Text GLabel 3350 30200 2    50   Input ~ 0
+Text GLabel 3400 30000 2    50   Input ~ 0
 COIL_T-
 Wire Wire Line
@@
 	1500 28550 1850 28550
 Wire Wire Line
-	1650 30300 1750 30300
+	1700 30100 1800 30100
 $Comp
 L power:+5V #PWR038
 U 1 1 5C83A002
-P 1650 29900
-F 0 "#PWR038" H 1650 29750 50  0001 C CNN
-F 1 "+5V" H 1665 30073 50  0000 C CNN
-F 2 "" H 1650 29900 50  0001 C CNN
-F 3 "" H 1650 29900 50  0001 C CNN
-	1    1650 29900
+P 1700 29700
+F 0 "#PWR038" H 1700 29550 50  0001 C CNN
+F 1 "+5V" H 1715 29873 50  0000 C CNN
+F 2 "" H 1700 29700 50  0001 C CNN
+F 3 "" H 1700 29700 50  0001 C CNN
+	1    1700 29700
 	1    0    0    -1
 $EndComp
 Wire Wire Line
-	1750 30000 1650 30000
+	1800 29800 1700 29800
 Wire Wire Line
-	1650 30000 1650 29900
+	1700 29800 1700 29700
 $Comp
 L power:-5V #PWR037
 U 1 1 5C83A00A
-P 1400 29900
-F 0 "#PWR037" H 1400 30000 50  0001 C CNN
-F 1 "-5V" H 1415 30073 50  0000 C CNN
-F 2 "" H 1400 29900 50  0001 C CNN
-F 3 "" H 1400 29900 50  0001 C CNN
-	1    1400 29900
+P 1450 29700
+F 0 "#PWR037" H 1450 29800 50  0001 C CNN
+F 1 "-5V" H 1465 29873 50  0000 C CNN
+F 2 "" H 1450 29700 50  0001 C CNN
+F 3 "" H 1450 29700 50  0001 C CNN
+	1    1450 29700
 	1    0    0    -1
 $EndComp
 Wire Wire Line
-	1400 29900 1400 30100
+	1450 29700 1450 29900
 Wire Wire Line
-	1400 30100 1750 30100
+	1450 29900 1800 29900
 Wire Wire Line
 	3250 28450 3350 28450
 Wire Wire Line
 	3250 28650 3350 28650
-Text GLabel 1650 30300 0    50   Input ~ 0
+Text GLabel 1700 30100 0    50   Input ~ 0
 DAC_OUT_COIL_T_CTRL
 $Comp
@@
 L power:GNDA #PWR039
 U 1 1 5CA9275F
-P 1650 30600
-F 0 "#PWR039" H 1650 30350 50  0001 C CNN
-F 1 "GNDA" H 1655 30427 50  0000 C CNN
-F 2 "" H 1650 30600 50  0001 C CNN
-F 3 "" H 1650 30600 50  0001 C CNN
-	1    1650 30600
+P 1700 30400
+F 0 "#PWR039" H 1700 30150 50  0001 C CNN
+F 1 "GNDA" H 1705 30227 50  0000 C CNN
+F 2 "" H 1700 30400 50  0001 C CNN
+F 3 "" H 1700 30400 50  0001 C CNN
+	1    1700 30400
 	1    0    0    -1
 $EndComp
 Wire Wire Line
-	1650 30600 1650 30500
+	1700 30400 1700 30300
 Wire Wire Line
-	1650 30500 1750 30500
+	1700 30300 1800 30300
 $Sheet
-S 1750 29900 1500 700
+S 1800 29700 1500 700
 U 5C839FF6
 F0 "Coil Current Source - Tracking" 50
 F1 "Coil_Current_Source.sch" 50
-F2 "DAC_IN" I L 1750 30300 50
-F3 "COIL+" O R 3250 30000 50
-F4 "COIL-" O R 3250 30200 50
-F5 "PWR_IN+" I L 1750 30000 50
-F6 "GND" U L 1750 30500 50
-F7 "PWR_IN-" I L 1750 30100 50
+F2 "DAC_IN" I L 1800 30100 50
+F3 "COIL+" O R 3300 29800 50
+F4 "COIL-" O R 3300 30000 50
+F5 "PWR_IN+" I L 1800 29800 50
+F6 "GND" U L 1800 30300 50
+F7 "PWR_IN-" I L 1800 29900 50
 $EndSheet
 Wire Wire Line
-	3250 30000 3350 30000
+	3300 29800 3400 29800
 Wire Wire Line
-	3250 30200 3350 30200
+	3300 30000 3400 30000
 $Sheet
 S 4050 19100 900  900
@@
 F 0 "U13" H 6750 18350 50  0000 C CNN
 F 1 "TBD" H 6800 18050 50  0000 C CNN
-F 2 "TBD" H 6550 18200 50  0001 C CNN
+F 2 "Sentisa-IC:SO-8" H 6550 18200 50  0001 C CNN
 F 3 "" H 6550 18200 50  0001 C CNN
 F 4 "TBD" H 6550 18200 50  0001 C CNN "MFR"
@@
 F 0 "U13" H 8300 18667 50  0000 C CNN
 F 1 "TBD" H 8300 18576 50  0000 C CNN
-F 2 "TBD" H 8300 18300 50  0001 C CNN
+F 2 "Sentisa-IC:SO-8" H 8300 18300 50  0001 C CNN
 F 3 "" H 8300 18300 50  0001 C CNN
 F 4 "TBD" H 8300 18300 50  0001 C CNN "MFR"
@@
 F 0 "U13" H 7358 19846 50  0000 L CNN
 F 1 "TBD" H 7358 19755 50  0000 L CNN
-F 2 "TBD" H 7400 19800 50  0001 C CNN
+F 2 "Sentisa-IC:SO-8" H 7400 19800 50  0001 C CNN
 F 3 "" H 7400 19800 50  0001 C CNN
 F 4 "TBD" H 7400 19800 50  0001 C CNN "MFR"
