File: uSensor_v1/uSensor_v1.sch (KiCad schematic (older format))
At the start: 224 parts, among them J1 +12V Supply, J2 Conn_01x03, J3 Conn_01x03, J4 NS25-W8P 6-pin 2,54mm, J5 USB_B, J6 GNDA-GNDD Jumper, J7 Barrel_Jack_Switch, Q1 BC817-25, Q2 BC817-25, SW1 SW_Push, SW2 SW_Push, SW3 SW_Push, U1 AM10TW-2405DZ, U10 KSS-213 Connector, U11 AD7795, U12 AD5667, U13 TBD, U15 REF192, U2 LD1117A, U22 RCLAMP, U3 STM32F407VGTx, U4 MCP9700AT, U5 MCP9700AT, U6 LM6132A, U7 MCP9700AT, U8 MCP9700AT, U9 UG-2864KSWLG01

Commit message: Review.
Parts:
- added C?: 100n 16V X5R, Capacitor_SMD:C_0603_1608Metric_Pad1.05x0.95mm_HandSolder, symbol Device:C
- added L?: 10u, symbol Device:L
Connections:
- net +3V3: now also L?.2; no longer U3.22 (VDDA)
- net GNDA: now also U3.20 (VSSA), C?.2
- net GNDD: no longer U3.20 (VSSA)
- new net: C?.1, L?.1, U3.22 (VDDA)
Other:
- moved on the sheet: C13, C16, C7, C8
Changed lines of the file:
@@
 	2200 7250 3100 7250
 Wire Wire Line
-	7200 12300 7100 12300
-Wire Wire Line
 	6800 12300 6800 12200
 Wire Wire Line
@@
 Wire Wire Line
 	7100 12200 7100 12300
-Connection ~ 7100 12300
 Wire Wire Line
 	7100 12300 7000 12300
-Wire Wire Line
-	7200 12200 7200 12300
 $Comp
 L Device:C C6
@@
 L power:+3V3 #PWR069
 U 1 1 647CDFB9
-P 10250 4800
-F 0 "#PWR069" H 10250 4650 50  0001 C CNN
-F 1 "+3V3" H 10265 4973 50  0000 C CNN
-F 2 "" H 10250 4800 50  0001 C CNN
-F 3 "" H 10250 4800 50  0001 C CNN
-	1    10250 4800
+P 10250 4450
+F 0 "#PWR069" H 10250 4300 50  0001 C CNN
+F 1 "+3V3" H 10265 4623 50  0000 C CNN
+F 2 "" H 10250 4450 50  0001 C CNN
+F 3 "" H 10250 4450 50  0001 C CNN
+	1    10250 4450
 	-1   0    0    -1
 $EndComp
@@
 L Device:C C7
 U 1 1 647CDFCD
-P 7850 5150
-F 0 "C7" H 7965 5196 50  0000 L CNN
-F 1 "100n 16V X5R" H 7965 5105 50  0000 L CNN
-F 2 "Capacitor_SMD:C_0603_1608Metric_Pad1.05x0.95mm_HandSolder" H 7888 5000 50  0001 C CNN
-F 3 "~" H 7850 5150 50  0001 C CNN
-	1    7850 5150
+P 7850 4800
+F 0 "C7" H 7965 4846 50  0000 L CNN
+F 1 "100n 16V X5R" H 7965 4755 50  0000 L CNN
+F 2 "Capacitor_SMD:C_0603_1608Metric_Pad1.05x0.95mm_HandSolder" H 7888 4650 50  0001 C CNN
+F 3 "~" H 7850 4800 50  0001 C CNN
+	1    7850 4800
 	-1   0    0    -1
 $EndComp
@@
 L Device:C C8
 U 1 1 647CDFD4
-P 8650 5150
-F 0 "C8" H 8765 5196 50  0000 L CNN
-F 1 "100n 16V X5R" H 8765 5105 50  0000 L CNN
-F 2 "Capacitor_SMD:C_0603_1608Metric_Pad1.05x0.95mm_HandSolder" H 8688 5000 50  0001 C CNN
-F 3 "~" H 8650 5150 50  0001 C CNN
-	1    8650 5150
+P 8650 4800
+F 0 "C8" H 8765 4846 50  0000 L CNN
+F 1 "100n 16V X5R" H 8765 4755 50  0000 L CNN
+F 2 "Capacitor_SMD:C_0603_1608Metric_Pad1.05x0.95mm_HandSolder" H 8688 4650 50  0001 C CNN
+F 3 "~" H 8650 4800 50  0001 C CNN
+	1    8650 4800
 	-1   0    0    -1
 $EndComp
@@
 L Device:C C13
 U 1 1 647CDFDB
-P 9450 5150
-F 0 "C13" H 9335 5196 50  0000 R CNN
-F 1 "100n 16V X5R" H 9335 5105 50  0000 R CNN
-F 2 "Capacitor_SMD:C_0603_1608Metric_Pad1.05x0.95mm_HandSolder" H 9488 5000 50  0001 C CNN
-F 3 "~" H 9450 5150 50  0001 C CNN
-	1    9450 5150
+P 9450 4800
+F 0 "C13" H 9335 4846 50  0000 R CNN
+F 1 "100n 16V X5R" H 9335 4755 50  0000 R CNN
+F 2 "Capacitor_SMD:C_0603_1608Metric_Pad1.05x0.95mm_HandSolder" H 9488 4650 50  0001 C CNN
+F 3 "~" H 9450 4800 50  0001 C CNN
+	1    9450 4800
 	1    0    0    -1
 $EndComp
@@
 Connection ~ 5200 5400
 Wire Wire Line
-	7850 5300 7850 5400
+	7850 4950 7850 5050
 Wire Wire Line
-	8650 5300 8650 5400
+	8650 4950 8650 5050
 Wire Wire Line
-	8650 5400 7850 5400
+	8650 5050 7850 5050
 Wire Wire Line
-	9450 5300 9450 5400
+	9450 4950 9450 5050
 Wire Wire Line
-	9450 5400 8650 5400
-Connection ~ 8650 5400
+	9450 5050 8650 5050
+Connection ~ 8650 5050
 Wire Wire Line
-	10250 5400 9450 5400
-Connection ~ 9450 5400
+	10250 5050 9450 5050
+Connection ~ 9450 5050
 Wire Wire Line
-	10250 4900 9450 4900
+	10250 4550 9450 4550
 Wire Wire Line
-	9450 4900 9450 5000
+	9450 4550 9450 4650
 Wire Wire Line
-	10250 4900 10250 4800
+	10250 4550 10250 4450
 Wire Wire Line
-	9450 4900 8650 4900
+	9450 4550 8650 4550
 Wire Wire Line
-	8650 4900 8650 5000
-Connection ~ 9450 4900
+	8650 4550 8650 4650
+Connection ~ 9450 4550
 Wire Wire Line
-	8650 4900 7850 4900
+	8650 4550 7850 4550
 Wire Wire Line
-	7850 4900 7850 5000
-Connection ~ 8650 4900
+	7850 4550 7850 4650
+Connection ~ 8650 4550
 Wire Wire Line
 	4400 4900 4400 5000
@@
 	7300 6200 7200 6200
 Connection ~ 7200 6200
-Wire Wire Line
-	7000 12400 7000 12300
 $Comp
 L Device:R R7
@@
 Wire Wire Line
 	6500 6100 6500 6200
-Wire Wire Line
-	7300 6200 7400 6200
-Wire Wire Line
-	7400 6200 7400 6300
-Connection ~ 7300 6200
 $Comp
 L Device:C C16
 U 1 1 647CE051
-P 10250 5150
-F 0 "C16" H 10135 5196 50  0000 R CNN
-F 1 "100n 16V X5R" H 10135 5105 50  0000 R CNN
-F 2 "Capacitor_SMD:C_0603_1608Metric_Pad1.05x0.95mm_HandSolder" H 10288 5000 50  0001 C CNN
-F 3 "~" H 10250 5150 50  0001 C CNN
-	1    10250 5150
+P 10250 4800
+F 0 "C16" H 10135 4846 50  0000 R CNN
+F 1 "100n 16V X5R" H 10135 4755 50  0000 R CNN
+F 2 "Capacitor_SMD:C_0603_1608Metric_Pad1.05x0.95mm_HandSolder" H 10288 4650 50  0001 C CNN
+F 3 "~" H 10250 4800 50  0001 C CNN
+	1    10250 4800
 	1    0    0    -1
 $EndComp
 Wire Wire Line
-	10250 5000 10250 4900
-Connection ~ 10250 4900
+	10250 4650 10250 4550
+Connection ~ 10250 4550
 Wire Wire Line
-	10250 5300 10250 5400
+	10250 4950 10250 5050
 Wire Wire Line
 	6500 5700 6700 5700
@@
 	1600 8850 1800 8850
 Wire Wire Line
-	7100 6200 7100 4900
+	7100 6200 7100 4550
 Wire Wire Line
-	7100 4900 7850 4900
+	7100 4550 7850 4550
 Connection ~ 7100 6200
-Connection ~ 7850 4900
+Connection ~ 7850 4550
 $Comp
 L power:+3V3 #PWR011
@@
 Connection ~ 4400 4900
 Wire Wire Line
-	10250 5500 10250 5400
-Connection ~ 10250 5400
+	10250 5150 10250 5050
+Connection ~ 10250 5050
 Wire Wire Line
 	4400 5500 4400 5400
@@
 L power:GNDD #PWR0130
 U 1 1 5D0C2B75
-P 7000 12400
-F 0 "#PWR0130" H 7000 12150 50  0001 C CNN
-F 1 "GNDD" H 7004 12245 50  0000 C CNN
-F 2 "" H 7000 12400 50  0001 C CNN
-F 3 "" H 7000 12400 50  0001 C CNN
-	1    7000 12400
+P 6800 12400
+F 0 "#PWR0130" H 6800 12150 50  0001 C CNN
+F 1 "GNDD" H 6804 12245 50  0000 C CNN
+F 2 "" H 6800 12400 50  0001 C CNN
+F 3 "" H 6800 12400 50  0001 C CNN
+	1    6800 12400
 	1    0    0    -1
 $EndComp
@@
 L power:GNDD #PWR0136
 U 1 1 5D0C7735
-P 10250 5500
-F 0 "#PWR0136" H 10250 5250 50  0001 C CNN
-F 1 "GNDD" H 10254 5345 50  0000 C CNN
-F 2 "" H 10250 5500 50  0001 C CNN
-F 3 "" H 10250 5500 50  0001 C CNN
-	1    10250 5500
+P 10250 5150
+F 0 "#PWR0136" H 10250 4900 50  0001 C CNN
+F 1 "GNDD" H 10254 4995 50  0000 C CNN
+F 2 "" H 10250 5150 50  0001 C CNN
+F 3 "" H 10250 5150 50  0001 C CNN
+	1    10250 5150
 	1    0    0    -1
 $EndComp
@@
 Wire Wire Line
 	9700 24350 9800 24350
+$Comp
+L Device:C C?
+U 1 1 5C83B3F6
+P 8000 5750
+F 0 "C?" H 7885 5796 50  0000 R CNN
+F 1 "100n 16V X5R" H 7885 5705 50  0000 R CNN
+F 2 "Capacitor_SMD:C_0603_1608Metric_Pad1.05x0.95mm_HandSolder" H 8038 5600 50  0001 C CNN
+F 3 "~" H 8000 5750 50  0001 C CNN
+	1    8000 5750
+	-1   0    0    -1
+$EndComp
+$Comp
+L Device:L L?
+U 1 1 5C981B92
+P 8250 5500
+F 0 "L?" V 8440 5500 50  0000 C CNN
+F 1 "10u" V 8349 5500 50  0000 C CNN
+F 2 "" H 8250 5500 50  0001 C CNN
+F 3 "~" H 8250 5500 50  0001 C CNN
+	1    8250 5500
+	0    -1   -1   0
+$EndComp
+$Comp
+L power:GNDA #PWR?
+U 1 1 5CA30877
+P 7200 12400
+F 0 "#PWR?" H 7200 12150 50  0001 C CNN
+F 1 "GNDA" H 7205 12227 50  0000 C CNN
+F 2 "" H 7200 12400 50  0001 C CNN
+F 3 "" H 7200 12400 50  0001 C CNN
+	1    7200 12400
+	1    0    0    -1
+$EndComp
+Wire Wire Line
+	6800 12400 6800 12300
+Connection ~ 6800 12300
+Wire Wire Line
+	7200 12400 7200 12200
+$Comp
+L power:GNDA #PWR?
+U 1 1 5CD5ED2C
+P 8000 6000
+F 0 "#PWR?" H 8000 5750 50  0001 C CNN
+F 1 "GNDA" H 8005 5827 50  0000 C CNN
+F 2 "" H 8000 6000 50  0001 C CNN
+F 3 "" H 8000 6000 50  0001 C CNN
+	1    8000 6000
+	1    0    0    -1
+$EndComp
+Wire Wire Line
+	8000 6000 8000 5900
+$Comp
+L power:+3V3 #PWR?
+U 1 1 5CE029A8
+P 8500 5400
+F 0 "#PWR?" H 8500 5250 50  0001 C CNN
+F 1 "+3V3" H 8515 5573 50  0000 C CNN
+F 2 "" H 8500 5400 50  0001 C CNN
+F 3 "" H 8500 5400 50  0001 C CNN
+	1    8500 5400
+	-1   0    0    -1
+$EndComp
+Wire Wire Line
+	8400 5500 8500 5500
+Wire Wire Line
+	8500 5500 8500 5400
+Wire Wire Line
+	8000 5600 8000 5500
+Wire Wire Line
+	8000 5500 8100 5500
+Wire Wire Line
+	7400 6300 7400 5500
+Wire Wire Line
+	7400 5500 8000 5500
+Connection ~ 8000 5500
 $EndSCHEMATC
