File: uSensor_v1/uSensor_v1.kicad_pcb (KiCad board)
At the start: 2 copper layers, 171 x 76.4 mm, 285 parts, among them J1 +12V Supply, J2 Conn_01x03, J3 Conn_01x03, J4 NS25-W8P 6-pin 2,54mm, J5 USB_B, J6 GNDA-GNDD Jumper, J7 Barrel_Jack_Switch, Q1 BC817-25, Q2 BC817-25, Q3 BC847PN-7-F, Q4 BC847PN-7-F, SW1 SW_Push, SW2 SW_Push, SW3 SW_Push, U1 AM10TW-2405DZ, U10 KSS-213 Connector, U11 AD7795, U12 AD5667, U13 TBD, U14 TBD, U15 REF192, U16 TBD, U17 TBD, U2 LD1117A, U22 RCLAMP, U3 STM32F407VGTx, U4 MCP9700AT, U5 MCP9700AT, U6 LM6132A, U7 MCP9700AT, U8 MCP9700AT, U9 UG-2864KSWLG01

Commit message: Layout in progress.
Parts:
- removed TP22: TP, Sentisa-Connectors:TestPoint_Probe_1.0mmDiameter_0.6mmDrill
- added CS1: Curr_Sens, Sentisa-Connectors:Current_Sense_Pin_Header_SMD_Pitch1.27mm, F.Cu at (168.4, 57.5)
- added CS2: Curr_Sens, Sentisa-Connectors:Current_Sense_Pin_Header_SMD_Pitch1.27mm, F.Cu at (168.4, 59.6)
- added CS3: Curr_Sens, Sentisa-Connectors:Current_Sense_Pin_Header_SMD_Pitch1.27mm, F.Cu at (160.1, 58.2)
- moved TP92 231.3 mm to (20.6, 73.5)
- moved TP97 225.3 mm to (18.5, 74.1)
- moved TP91 224.5 mm to (16.4, 73.4)
- moved TP94 222.4 mm to (23.7, 73.7)
- moved TP1 221.0 mm to (23.9, 40.8)
- moved TP98 217.8 mm to (21.8, 77.7)
- moved TP93 217.7 mm to (19.5, 76.6)
- moved TP96 214.8 mm to (21.6, 75.2)
- moved TP95 213.7 mm to (17.5, 75.7)
- moved TP85 203.1 mm to (72.4, 23.4)
- moved TP87 202.5 mm to (74.8, 23.4)
- moved TP88 200.5 mm to (75.2, 25.7)
- moved TP27 197.2 mm to (55.4, 74.0)
- moved TP89 193.5 mm to (72.5, 25.1)
- moved TP20 193.5 mm to (70.2, 25.2)
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Connections:
- L4 pad 1: SENS_LD -> Net-(CS3-Pad2)
- TP21 pad 1: Net-(R9-Pad1) -> DAC_~LDAC
- U10 pad 13: COIL_F+ -> Net-(CS1-Pad2)
- U10 pad 14: COIL_T+ -> Net-(CS2-Pad2)
- U12 pad 1: DAC_OUT_COIL_T_CTRL -> DAC_OUT_COIL_F_CTRL
- U12 pad 2: DAC_OUT_COIL_F_CTRL -> DAC_OUT_COIL_T_CTRL
- U3 pad 66: ADC_~CS -> Net-(U3-Pad66)
- U3 pad 77: Net-(U3-Pad77) -> ADC_~CS
Routing:
- net ADC_~CS: track 7.31 -> 141.2 mm, vias 0 -> 3
- net ADC_SCLK: track 4.07 -> 136.1 mm, vias 0 -> 3
- net ADC_DOUT: track 6.22 -> 128.9 mm, vias 0 -> 3
- net ADC_DIN: track 4.07 -> 123.3 mm, vias 0 -> 3
- net DAC_OUT_COIL_T_CTRL: track 0.00 -> 93.2 mm, vias 0 -> 1
- net DAC_OUT_COIL_F_CTRL: track 0.00 -> 89.7 mm, vias 0 -> 1
- net DAC_~LDAC: track 3.79 -> 85.2 mm, vias 0 -> 1
- net DAC_~CLR: track 0.00 -> 77.8 mm, vias 0 -> 1
- net SENS_PD: track 0.00 -> 75.6 mm, vias 0 -> 2
- net DAC_ADDR: track 0.00 -> 74.5 mm, vias 0 -> 1
- net +5V: track 62.9 -> 129.5 mm
- net TEMP_SENS_OUT_4: track 0.00 -> 63.3 mm, vias 0 -> 3
- net TEMP_SENS_OUT_3: track 0.00 -> 59.0 mm, vias 0 -> 3
- net DAC_SCL: track 0.00 -> 58.5 mm, vias 0 -> 2
- net DAC_SDA: track 0.00 -> 57.4 mm, vias 0 -> 2
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- added copper zone on B.Cu, net GNDA
- added copper zone on B.Cu, net GNDD

Commit message: Layout improving.
Parts:
- moved TP20 0.54 mm to (70.0, 25.7)
Changed lines of the file:
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@@
   )
   (module Sentisa-Connectors:TestPoint_Probe_1.0mmDiameter_0.6mmDrill (layer F.Cu)
-    (at 70.2 25.2)
+    (at 70 25.7)
     (tags TestPoint_Probe_1.0mmDiameter_0.6mmDrill)
     (fp_text reference TP20 (at 0 -1.5) (layer F.SilkS)

Commit message: Layout in progress.
Parts:
- moved C56 14.1 mm to (162.4, 38.7)
- moved J2 14.1 mm to (165.9, 69.9)
- moved R27 14.1 mm to (175.2, 39.2)
- moved R74 14.1 mm to (165.9, 64.9)
- moved TP35 14.1 mm to (176.5, 71.4)
- moved TP38 14.1 mm to (173.5, 71.4)
- moved TP41 14.1 mm to (172.4, 33.7)
- moved TP56 14.1 mm to (172.6, 39.2)
- moved C1 14.1 mm to (154.6, 79.8)
- moved C19 14.1 mm to (153.1, 83.7)
- moved C29 14.1 mm to (180.8, 56.1)
- moved C30 14.1 mm to (180.8, 54.3)
- moved C31 14.1 mm to (151.9, 59.0)
- moved C32 14.1 mm to (152.7, 61.0)
- moved C33 14.1 mm to (152.7, 62.7)
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Routing:
- net +5V: track 129.5 -> 299.2 mm, vias 0 -> 6
- net +3V3: track 113.9 -> 171.8 mm, vias 1 -> 12
- net GNDA: track 0.00 -> 25.4 mm
- net DAC_LD_CTRL: track 1.91 -> 26.9 mm, vias 0 -> 1
- net LCD_SI: track 65.9 -> 70.1 mm
- net SWITCH_1: track 80.3 -> 76.3 mm
- net -5V: track 28.1 -> 24.8 mm
- net ADC_SCLK: track 136.1 -> 133.2 mm
- net LCD_A0: track 68.6 -> 71.1 mm
- net LCD_CS: track 70.6 -> 73.0 mm
- net LCD_RST: track 72.4 -> 74.8 mm
- net TEMP_SENS_OUT_1: track 53.2 -> 55.5 mm
- net SENS_PD_ADC: track 18.7 -> 20.9 mm, vias 0 -> 1
- net TEMP_SENS_OUT_2: track 56.9 -> 59.0 mm
- net ADC_DOUT: track 128.9 -> 127.0 mm
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Other:
- board size 171 x 76.4 mm -> 180 x 81.4 mm

Commit message: Layout in progress.
Parts:
- moved TP44 40.0 mm to (138.8, 36.9)
- moved C29 36.6 mm to (145.3, 47.3)
- moved C30 36.6 mm to (145.3, 45.5)
- moved TP68 36.5 mm to (127.3, 38.1)
- moved C58 36.5 mm to (123.3, 38.2)
- moved R1 36.5 mm to (119.8, 84.2)
- moved R2 36.5 mm to (119.8, 85.9)
- moved R3 36.5 mm to (119.8, 82.5)
- moved TP46 36.5 mm to (123.8, 57.5)
- moved TP47 36.5 mm to (127.8, 57.5)
- moved TP48 36.5 mm to (119.8, 57.5)
- moved TP49 36.5 mm to (121.8, 57.5)
- moved TP72 36.5 mm to (117.8, 61.4)
- moved TP78 36.5 mm to (121.8, 69.8)
- moved TP99 36.5 mm to (125.8, 57.5)
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Routing:
- net +3V3: track 171.8 -> 246.1 mm, vias 12 -> 13
- net DAC_OUT_COIL_F_CTRL: track 88.4 -> 45.1 mm
- net DAC_OUT_COIL_T_CTRL: track 91.9 -> 49.7 mm
- net ADC_~CS: track 139.4 -> 98.5 mm
- net ADC_SCLK: track 133.2 -> 93.3 mm
- net ADC_DOUT: track 127.0 -> 95.1 mm
- net ADC_DIN: track 121.4 -> 90.4 mm
- net SENS_D: track 60.0 -> 53.7 mm
- net +5V: track 299.2 -> 295.3 mm
- net SENS_B: track 72.8 -> 69.0 mm
- net Net-(C26-Pad1): track 19.2 -> 16.3 mm
- net Net-(RV1-Pad2): track 12.0 -> 9.40 mm
- net Net-(C25-Pad2): track 13.6 -> 15.5 mm
- net Net-(C35-Pad1): track 11.6 -> 13.5 mm
- net Net-(TP34-Pad1): track 11.4 -> 9.55 mm
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Other:
- board size 180 x 81.4 mm -> 145.5 x 81.4 mm

Commit message: Layout in progress.
Parts:
- moved J6 18.1 mm to (101.0, 37.4), turned to 270 degrees
- moved TP59 14.4 mm to (142.1, 17.6)
- moved TP38 8.05 mm to (130.2, 61.1)
- moved C19 7.91 mm to (109.7, 75.1), turned to 90 degrees
- moved TP35 7.90 mm to (133.1, 62.9)
- moved C29 7.90 mm to (137.4, 47.3)
- moved C30 7.90 mm to (137.4, 45.5)
- moved C31 7.90 mm to (108.5, 50.7)
- moved C32 7.90 mm to (109.3, 52.7)
- moved C33 7.90 mm to (109.3, 54.4)
- moved C34 7.90 mm to (108.5, 56.4)
- moved C42 7.90 mm to (137.6, 54.6)
- moved C43 7.90 mm to (141.9, 33.8)
- moved C45 7.90 mm to (141.5, 26.0)
- moved C46 7.90 mm to (122.5, 47.6)
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Routing:
- net +5V: track 295.3 -> 525.7 mm, vias 6 -> 22
- net -5V: track 24.8 -> 220.5 mm, vias 0 -> 24
- net SENS_PD_ADC: track 22.4 -> 112.0 mm, vias 1 -> 3
- net DAC_LD_CTRL: track 26.6 -> 84.1 mm, vias 1 -> 3
- net TEMP_SENS_OUT_4: track 65.1 -> 49.8 mm
- net DAC_OUT_COIL_F_CTRL: track 45.1 -> 59.9 mm
- net DAC_OUT_COIL_T_CTRL: track 49.7 -> 64.4 mm
- net TEMP_SENS_OUT_3: track 60.9 -> 49.6 mm
- net ADC_~CS: track 98.5 -> 107.5 mm
- net TEMP_SENS_OUT_2: track 59.0 -> 50.1 mm
- net ADC_SCLK: track 93.3 -> 101.7 mm
- net TEMP_SENS_OUT_1: track 55.5 -> 50.1 mm
- net +3V3: track 246.1 -> 249.9 mm, vias 13 -> 15
- net REF_2.5V: track 127.0 -> 126.2 mm
- net GNDD: vias 0 -> 6
Other:
- board size 145.5 x 81.4 mm -> 137.6 x 77.4 mm

Commit message: Connection done.
Parts:
- moved C23 51.9 mm to (142.7, 68.5)
- moved U7 51.8 mm to (139.9, 68.5)
- moved U5 50.5 mm to (137.7, 23.2), turned to 180 degrees
- moved C22 47.0 mm to (137.8, 26.0), turned to 180 degrees
- moved C21 23.5 mm to (113.5, 66.9)
- moved U4 23.5 mm to (110.8, 66.9)
- moved C24 20.6 mm to (111.5, 28.8)
- moved U8 20.5 mm to (108.7, 28.8)
- moved TP26 9.46 mm to (89.5, 49.0)
- moved TP36 8.81 mm to (131.8, 72.0)
- moved TP73 8.27 mm to (123.6, 86.0)
- moved TP24 7.36 mm to (89.5, 51.0)
- moved TP25 5.16 mm to (89.5, 53.0)
- moved TP70 5.02 mm to (123.6, 84.0)
- moved TP83 3.98 mm to (109.9, 63.2)
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Connections:
- C21 pad 1: +3V3 -> +5V
- C21 pad 2: GNDD -> GNDA
- C22 pad 1: +3V3 -> +5V
- C22 pad 2: GNDD -> GNDA
- C23 pad 1: +3V3 -> +5V
- C23 pad 2: GNDD -> GNDA
- C24 pad 1: +3V3 -> +5V
- C24 pad 2: GNDD -> GNDA
- U4 pad 1: +3V3 -> +5V
- U4 pad 2: TEMP_SENS_OUT_1 -> TEMP_SENS_OUT_2
- U4 pad 3: GNDD -> GNDA
- U5 pad 1: +3V3 -> +5V
- U5 pad 3: GNDD -> GNDA
- U7 pad 1: +3V3 -> +5V
- U7 pad 2: TEMP_SENS_OUT_2 -> TEMP_SENS_OUT_1
- U7 pad 3: GNDD -> GNDA
- U8 pad 1: +3V3 -> +5V
- U8 pad 3: GNDD -> GNDA
Routing:
- net TEMP_SENS_OUT_1: track 50.1 -> 143.2 mm, vias 3 -> 5
- net TEMP_SENS_OUT_3: track 49.6 -> 127.7 mm, vias 3 -> 6
- net REF_2.5V: track 126.2 -> 185.4 mm, vias 0 -> 8
- net TEMP_SENS_OUT_4: track 49.8 -> 84.5 mm
- net TEMP_SENS_OUT_2: track 50.1 -> 79.7 mm
- net +5V: track 525.7 -> 544.4 mm
- net +3V3: track 249.9 -> 267.9 mm, vias 15 -> 21
- net COIL_T-: track 24.9 -> 31.8 mm
- net Net-(J3-Pad3): track 9.19 -> 15.1 mm
- net Net-(C1-Pad1): track 12.5 -> 14.0 mm
- net /SENS_IN_AMP_CH_A_B/SENS_OUT_2: track 25.4 -> 24.1 mm
- net Net-(C1-Pad2): track 6.78 -> 7.99 mm
- net SENS_B: track 69.0 -> 70.2 mm
- net SENS_PD_ADC: track 112.0 -> 112.7 mm
- net Net-(C50-Pad2): track 8.91 -> 8.29 mm
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
Commit message: Layout ready to 1st review.
Parts:
- J1: footprint Connector_PinHeader_2.54mm:PinHeader_1x02_P2.54mm_Vertical -> Connector_Molex:Molex_KK-254_AE-6410-02A_1x02_P2.54mm_Vertical
- moved TP87 91.9 mm to (143.5, 85.5)
- moved TP98 80.6 mm to (90.4, 37.5)
- moved TP93 79.5 mm to (97.5, 74.7)
- moved TP95 78.6 mm to (97.6, 54.6)
- moved TP20 70.6 mm to (106.7, 86.8)
- moved TP91 70.5 mm to (92.5, 61.6)
- moved TP88 65.5 mm to (140.6, 17.0)
- moved TP90 65.1 mm to (134.7, 35.6)
- moved TP85 58.3 mm to (127.6, 44.1)
- moved TP84 57.6 mm to (106.9, 67.8)
- moved TP94 51.0 mm to (72.6, 81.3)
- moved TP96 40.5 mm to (46.4, 44.0)
- moved TP97 39.6 mm to (22.9, 34.5)
- moved TP89 37.9 mm to (102.9, 48.9)
- moved TP86 30.2 mm to (105.2, 20.3)
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Routing:
- net Net-(D1-Pad2): track 14.2 -> 36.6 mm
- net REF_2.5V: track 185.4 -> 178.8 mm, vias 8 -> 4
- net Net-(C11-Pad2): track 48.6 -> 55.1 mm
- net -5V: track 221.1 -> 214.8 mm, vias 24 -> 22
- net +5V: track 544.4 -> 539.2 mm
- net TEMP_SENS_OUT_1: track 143.2 -> 138.1 mm, vias 5 -> 4
- net +3V3: track 267.9 -> 272.1 mm, vias 21 -> 22
- net SENS_A: track 63.5 -> 64.4 mm
- net DAC_OUT_COIL_T_CTRL: track 64.4 -> 63.7 mm
- net DAC_OUT_COIL_F_CTRL: track 59.9 -> 59.3 mm
- net TEMP_SENS_OUT_3: track 127.7 -> 127.4 mm, vias 6 -> 5
- net TEMP_SENS_OUT_4: vias 3 -> 2
- net TEMP_SENS_OUT_2: vias 3 -> 2
